File: SwitchMatrix_Design.sch (KiCad schematic (older format))
At the start: 180 parts, among them K1 ESC, K10 F8, K11 F9, K12 F10, K13 F11, K14 F12, K15 SW_Push, K16 SW_Push, K17 SW_Push, K18 SW_Push, K19 SW_Push, K2 F1, K20 SW_Push, K21 SW_Push, K22 SW_Push, K23 SW_Push, K24 SW_Push, K25 SW_Push, K26 SW_Push, K27 SW_Push, K28 SW_Push, K29 SW_Push, K3 F2, K30 SW_Push, K31 SW_Push, K32 SW_Push, K33 SW_Push, K34 SW_Push, K35 SW_Push, K36 SW_Push, K37 SW_Push, K38 SW_Push, K39 SW_Push, K4 F3, K40 SW_Push, K41 SW_Push, K42 SW_Push, K43 SW_Push, K44 SW_Push, K45 SW_Push, K46 SW_Push, K47 SW_Push, K48 SW_Push, K49 SW_Push, K5 F4, K50 SW_Push, K51 SW_Push, K52 SW_Push, K53 SW_Push, K54 SW_Push, K55 SW_Push, K56 SW_Push, K57 SW_Push, K58 SW_Push, K59 SW_Push, K6 F5, K60 SW_Push, K61 SW_Push, K62 SW_Push, K63 SW_Push, K64 SW_Push, K65 SW_Push, K66 SW_Push, K67 SW_Push, K68 SW_Push, K69 SW_Push, K7 F6, K70 SW_Push, K71 SW_Push, K72 SW_Push, K73 SW_Push, K74 SW_Push, K75 SW_Push, K76 SW_Push, K77 SW_Push, K78 SW_Push, K79 SW_Push, K8 Xevid, K80 SW_Push, K81 SW_Push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

Commit message: v1b2.6
Switch matrix annotated.
Parts:
- K15: value SW_Push -> KU1
- K16: value SW_Push -> PrtSc
- K17: value SW_Push -> PauseBrk
- K18: value SW_Push -> CDE
- K19: value SW_Push -> #1
- K20: value SW_Push -> #2
- K21: value SW_Push -> #3
- K22: value SW_Push -> #4
- K23: value SW_Push -> #5
- K24: value SW_Push -> #6
- K25: value SW_Push -> #7
- K26: value SW_Push -> #8
- K27: value SW_Push -> #9
- K28: value SW_Push -> #0
- K29: value SW_Push -> -
- K30: value SW_Push -> =
- K31: value SW_Push -> Backspace
- K32: value SW_Push -> Insert
- K33: value SW_Push -> PgUP
- K34: value SW_Push -> Tab
- K35: value SW_Push -> Q
- K36: value SW_Push -> W
- K37: value SW_Push -> E
- K38: value SW_Push -> R
- K39: value SW_Push -> T
- K40: value SW_Push -> Y
- K41: value SW_Push -> U
- K42: value SW_Push -> I
- K43: value SW_Push -> O
- K44: value SW_Push -> P
- K45: value SW_Push -> [
- K46: value SW_Push -> ]
- K47: value SW_Push -> Enter
- K48: value SW_Push -> Delete
- K49: value SW_Push -> PgDn
- K50: value SW_Push -> CpsLck
- K51: value SW_Push -> A
- K52: value SW_Push -> S
- K53: value SW_Push -> D
- K54: value SW_Push -> F
- K55: value SW_Push -> G
- K56: value SW_Push -> H
- K57: value SW_Push -> J
- K58: value SW_Push -> K
- K59: value SW_Push -> L
- K60: value SW_Push -> ;
- K61: value SW_Push -> '
- K62: value SW_Push -> #
- K63: value SW_Push -> Home
- K64: value SW_Push -> End
- K65: value SW_Push -> Shift
- K66: value SW_Push -> \\
- K67: value SW_Push -> Z
- K68: value SW_Push -> X
- K69: value SW_Push -> C
- K70: value SW_Push -> V
- K71: value SW_Push -> B
- K72: value SW_Push -> N
- K73: value SW_Push -> M
- K74: value SW_Push -> <
- K75: value SW_Push -> >
- K76: value SW_Push -> /
- K77: value SW_Push -> Shit
- K78: value SW_Push -> UpArrow
- K79: value SW_Push -> KU2
- K80: value SW_Push -> KU3
- K81, K86: value SW_Push -> Ctrl
- K82: value SW_Push -> Win
- K83: value SW_Push -> Alt
- K84: value SW_Push -> Space_Bar
- K85: value SW_Push -> AltGr
- K87: value SW_Push -> LeftArrow
- K88: value SW_Push -> DownArrow
- K89: value SW_Push -> RightArrow
- K90: value SW_Push -> KU4
