File: X95X/untitled.kicad_sch (KiCad schematic)
At the start: 182 parts, among them SW1 ESC, SW10 SW_Push, SW11 SW_Push, SW12 SW_Push, SW13 SW_Push, SW14 SW_Push, SW15 SW_Push, SW16 SW_Push, SW17 SW_Push, SW18 SW_Push, SW19 SW_Push, SW2 F1, SW20 SW_Push, SW21 SW_Push, SW22 SW_Push, SW23 SW_Push, SW24 SW_Push, SW25 SW_Push, SW26 SW_Push, SW27 SW_Push, SW28 SW_Push, SW29 SW_Push, SW3 F2, SW30 SW_Push, SW31 SW_Push, SW32 SW_Push, SW33 SW_Push, SW34 SW_Push, SW35 SW_Push, SW36 SW_Push, SW37 SW_Push, SW38 SW_Push, SW39 SW_Push, SW4 SW_Push, SW40 SW_Push, SW41 SW_Push, SW42 SW_Push, SW43 SW_Push, SW44 SW_Push, SW45 SW_Push, SW46 SW_Push, SW47 SW_Push, SW48 SW_Push, SW49 SW_Push, SW5 SW_Push, SW50 SW_Push, SW51 SW_Push, SW52 SW_Push, SW53 SW_Push, SW54 SW_Push, SW55 SW_Push, SW56 SW_Push, SW57 SW_Push, SW58 SW_Push, SW59 SW_Push, SW6 SW_Push, SW60 SW_Push, SW61 SW_Push, SW62 SW_Push, SW63 SW_Push, SW64 SW_Push, SW65 SW_Push, SW66 SW_Push, SW67 SW_Push, SW68 SW_Push, SW69 SW_Push, SW7 SW_Push, SW70 SW_Push, SW71 SW_Push, SW72 SW_Push, SW73 SW_Push, SW74 SW_Push, SW75 SW_Push, SW76 SW_Push, SW77 SW_Push, SW78 SW_Push, SW79 SW_Push, SW8 SW_Push, SW80 SW_Push, SW81 SW_Push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

Commit message: v.7c
Parts:
- removed D18, D19, D20, D21, D22, D23, D24, D25, D26, D27, D28, D29, D30, D31, D32, D33, D34, D51, D52, D53, D54, D55, D56, D57, D58, D59, D60, D61, D62, D63, D64, D65, D66, D83, D84, D85, D86, D87, D88, D89, D90, D91: D_Small, symbol Device:D_Small
- added D100, D101, D102, D103, D104, D105, D106, D107, D108, D109, D110, D111, D112, D113, D129, D130, D131, D132, D133, D134, D135, D136, D137, D138, D139, D140, D141, D142, D143, D144, D161, D162, D163, D164, D165, D166, D167, D168, D169, D170, D171, D99: D_Small, symbol Device:D_Small
- added D114: CapsLockRGB, LED_SMD:LED_SK6812MINI_PLCC4_3.5x3.5mm_P1.75mm, symbol LED:SK6812MINI
- added D115: ARGB, LED_SMD:LED_SK6812MINI_PLCC4_3.5x3.5mm_P1.75mm, symbol LED:SK6812MINI
- added D116: SRGB, LED_SMD:LED_SK6812MINI_PLCC4_3.5x3.5mm_P1.75mm, symbol LED:SK6812MINI
- added D117: DRGB, LED_SMD:LED_SK6812MINI_PLCC4_3.5x3.5mm_P1.75mm, symbol LED:SK6812MINI
- added D118: FRGB, LED_SMD:LED_SK6812MINI_PLCC4_3.5x3.5mm_P1.75mm, symbol LED:SK6812MINI
- added D119: GRGB, LED_SMD:LED_SK6812MINI_PLCC4_3.5x3.5mm_P1.75mm, symbol LED:SK6812MINI
- added D120: HRGB, LED_SMD:LED_SK6812MINI_PLCC4_3.5x3.5mm_P1.75mm, symbol LED:SK6812MINI
- added D121: JRGB, LED_SMD:LED_SK6812MINI_PLCC4_3.5x3.5mm_P1.75mm, symbol LED:SK6812MINI
- added D122: KRGB, LED_SMD:LED_SK6812MINI_PLCC4_3.5x3.5mm_P1.75mm, symbol LED:SK6812MINI
- added D123: LRGB, LED_SMD:LED_SK6812MINI_PLCC4_3.5x3.5mm_P1.75mm, symbol LED:SK6812MINI
- added D124: ;RGB, LED_SMD:LED_SK6812MINI_PLCC4_3.5x3.5mm_P1.75mm, symbol LED:SK6812MINI
- added D125: '@RGB, LED_SMD:LED_SK6812MINI_PLCC4_3.5x3.5mm_P1.75mm, symbol LED:SK6812MINI
- added D126: #~RGB, LED_SMD:LED_SK6812MINI_PLCC4_3.5x3.5mm_P1.75mm, symbol LED:SK6812MINI
- added D127: HomeRGB, LED_SMD:LED_SK6812MINI_PLCC4_3.5x3.5mm_P1.75mm, symbol LED:SK6812MINI
- added D128: EndRGB, LED_SMD:LED_SK6812MINI_PLCC4_3.5x3.5mm_P1.75mm, symbol LED:SK6812MINI
- added D145: LShift, LED_SMD:LED_SK6812MINI_PLCC4_3.5x3.5mm_P1.75mm, symbol LED:SK6812MINI
- added D146: \|RGB, LED_SMD:LED_SK6812MINI_PLCC4_3.5x3.5mm_P1.75mm, symbol LED:SK6812MINI
- added D147: ZRGB, LED_SMD:LED_SK6812MINI_PLCC4_3.5x3.5mm_P1.75mm, symbol LED:SK6812MINI
- added D148: XRGB, LED_SMD:LED_SK6812MINI_PLCC4_3.5x3.5mm_P1.75mm, symbol LED:SK6812MINI
- added D149: CRGB, LED_SMD:LED_SK6812MINI_PLCC4_3.5x3.5mm_P1.75mm, symbol LED:SK6812MINI
- added D150: VRGB, LED_SMD:LED_SK6812MINI_PLCC4_3.5x3.5mm_P1.75mm, symbol LED:SK6812MINI
- added D151: BRGB, LED_SMD:LED_SK6812MINI_PLCC4_3.5x3.5mm_P1.75mm, symbol LED:SK6812MINI
- added D152: NRGB, LED_SMD:LED_SK6812MINI_PLCC4_3.5x3.5mm_P1.75mm, symbol LED:SK6812MINI
- added D153: MRGB, LED_SMD:LED_SK6812MINI_PLCC4_3.5x3.5mm_P1.75mm, symbol LED:SK6812MINI
- added D154: ,<RGB, LED_SMD:LED_SK6812MINI_PLCC4_3.5x3.5mm_P1.75mm, symbol LED:SK6812MINI
- added D155: .>RGB, LED_SMD:LED_SK6812MINI_PLCC4_3.5x3.5mm_P1.75mm, symbol LED:SK6812MINI
- added D156: /?RGB, LED_SMD:LED_SK6812MINI_PLCC4_3.5x3.5mm_P1.75mm, symbol LED:SK6812MINI
- added D157: RShiftRGB, LED_SMD:LED_SK6812MINI_PLCC4_3.5x3.5mm_P1.75mm, symbol LED:SK6812MINI
- added D158: UpArrowRGB, LED_SMD:LED_SK6812MINI_PLCC4_3.5x3.5mm_P1.75mm, symbol LED:SK6812MINI
- added D159: U2RGB, LED_SMD:LED_SK6812MINI_PLCC4_3.5x3.5mm_P1.75mm, symbol LED:SK6812MINI
- added D160: U3RGB, LED_SMD:LED_SK6812MINI_PLCC4_3.5x3.5mm_P1.75mm, symbol LED:SK6812MINI
- added D172: LCtrlRGB, LED_SMD:LED_SK6812MINI_PLCC4_3.5x3.5mm_P1.75mm, symbol LED:SK6812MINI
- added D173: WinRGB, LED_SMD:LED_SK6812MINI_PLCC4_3.5x3.5mm_P1.75mm, symbol LED:SK6812MINI
- added D174: AltRGB, LED_SMD:LED_SK6812MINI_PLCC4_3.5x3.5mm_P1.75mm, symbol LED:SK6812MINI
- added D175: SpaceRGB, LED_SMD:LED_SK6812MINI_PLCC4_3.5x3.5mm_P1.75mm, symbol LED:SK6812MINI
- added D176: AltGrRGB, LED_SMD:LED_SK6812MINI_PLCC4_3.5x3.5mm_P1.75mm, symbol LED:SK6812MINI
- added D177: FnRGB, LED_SMD:LED_SK6812MINI_PLCC4_3.5x3.5mm_P1.75mm, symbol LED:SK6812MINI
- added D178: RCtrlRGB, LED_SMD:LED_SK6812MINI_PLCC4_3.5x3.5mm_P1.75mm, symbol LED:SK6812MINI
- added D179: LeftArrowRGB, LED_SMD:LED_SK6812MINI_PLCC4_3.5x3.5mm_P1.75mm, symbol LED:SK6812MINI
- added D18: ESCRGB, LED_SMD:LED_SK6812MINI_PLCC4_3.5x3.5mm_P1.75mm, symbol LED:SK6812MINI
- added D180: DownArrowRGB, LED_SMD:LED_SK6812MINI_PLCC4_3.5x3.5mm_P1.75mm, symbol LED:SK6812MINI
- added D181: RightArrowRGB, LED_SMD:LED_SK6812MINI_PLCC4_3.5x3.5mm_P1.75mm, symbol LED:SK6812MINI
- added D182: U4RGB, LED_SMD:LED_SK6812MINI_PLCC4_3.5x3.5mm_P1.75mm, symbol LED:SK6812MINI
- added D19: F1RGB, LED_SMD:LED_SK6812MINI_PLCC4_3.5x3.5mm_P1.75mm, symbol LED:SK6812MINI
- added D20: F2RGB, LED_SMD:LED_SK6812MINI_PLCC4_3.5x3.5mm_P1.75mm, symbol LED:SK6812MINI
- added D21: F3RGB, LED_SMD:LED_SK6812MINI_PLCC4_3.5x3.5mm_P1.75mm, symbol LED:SK6812MINI
- added D22: F4RGB, LED_SMD:LED_SK6812MINI_PLCC4_3.5x3.5mm_P1.75mm, symbol LED:SK6812MINI
- added D23: F5RGB, LED_SMD:LED_SK6812MINI_PLCC4_3.5x3.5mm_P1.75mm, symbol LED:SK6812MINI
- added D24: F6RGB, LED_SMD:LED_SK6812MINI_PLCC4_3.5x3.5mm_P1.75mm, symbol LED:SK6812MINI
- added D25: XEVRGB, LED_SMD:LED_SK6812MINI_PLCC4_3.5x3.5mm_P1.75mm, symbol LED:SK6812MINI
- added D26: F7RGB, LED_SMD:LED_SK6812MINI_PLCC4_3.5x3.5mm_P1.75mm, symbol LED:SK6812MINI
- added D27: F8RGB, LED_SMD:LED_SK6812MINI_PLCC4_3.5x3.5mm_P1.75mm, symbol LED:SK6812MINI
- added D28: F9RGB, LED_SMD:LED_SK6812MINI_PLCC4_3.5x3.5mm_P1.75mm, symbol LED:SK6812MINI
- added D29: F10RGB, LED_SMD:LED_SK6812MINI_PLCC4_3.5x3.5mm_P1.75mm, symbol LED:SK6812MINI
- added D30: F11RGB, LED_SMD:LED_SK6812MINI_PLCC4_3.5x3.5mm_P1.75mm, symbol LED:SK6812MINI
- added D31: F12RGB, LED_SMD:LED_SK6812MINI_PLCC4_3.5x3.5mm_P1.75mm, symbol LED:SK6812MINI
- added D32: U1RGB, LED_SMD:LED_SK6812MINI_PLCC4_3.5x3.5mm_P1.75mm, symbol LED:SK6812MINI
- added D33: PrtScRGB, LED_SMD:LED_SK6812MINI_PLCC4_3.5x3.5mm_P1.75mm, symbol LED:SK6812MINI
- added D34: PauseBrRGB, LED_SMD:LED_SK6812MINI_PLCC4_3.5x3.5mm_P1.75mm, symbol LED:SK6812MINI
- added D51: `RGB, LED_SMD:LED_SK6812MINI_PLCC4_3.5x3.5mm_P1.75mm, symbol LED:SK6812MINI
- added D52: 1RGB, LED_SMD:LED_SK6812MINI_PLCC4_3.5x3.5mm_P1.75mm, symbol LED:SK6812MINI
- added D53: 2RGB, LED_SMD:LED_SK6812MINI_PLCC4_3.5x3.5mm_P1.75mm, symbol LED:SK6812MINI
- added D54: 3RGB, LED_SMD:LED_SK6812MINI_PLCC4_3.5x3.5mm_P1.75mm, symbol LED:SK6812MINI
- added D55: 4RGB, LED_SMD:LED_SK6812MINI_PLCC4_3.5x3.5mm_P1.75mm, symbol LED:SK6812MINI
- added D56: 5RGB, LED_SMD:LED_SK6812MINI_PLCC4_3.5x3.5mm_P1.75mm, symbol LED:SK6812MINI
- added D57: 6RGB, LED_SMD:LED_SK6812MINI_PLCC4_3.5x3.5mm_P1.75mm, symbol LED:SK6812MINI
- added D58: 7RGB, LED_SMD:LED_SK6812MINI_PLCC4_3.5x3.5mm_P1.75mm, symbol LED:SK6812MINI
- added D59: 8RGB, LED_SMD:LED_SK6812MINI_PLCC4_3.5x3.5mm_P1.75mm, symbol LED:SK6812MINI
- added D60: 9RGB, LED_SMD:LED_SK6812MINI_PLCC4_3.5x3.5mm_P1.75mm, symbol LED:SK6812MINI
- added D61: 0RGB, LED_SMD:LED_SK6812MINI_PLCC4_3.5x3.5mm_P1.75mm, symbol LED:SK6812MINI
- added D62: -RGB, LED_SMD:LED_SK6812MINI_PLCC4_3.5x3.5mm_P1.75mm, symbol LED:SK6812MINI
- added D63: =RGB, LED_SMD:LED_SK6812MINI_PLCC4_3.5x3.5mm_P1.75mm, symbol LED:SK6812MINI
- added D64: BackSpaceRGB, LED_SMD:LED_SK6812MINI_PLCC4_3.5x3.5mm_P1.75mm, symbol LED:SK6812MINI
- added D65: InsertRGB, LED_SMD:LED_SK6812MINI_PLCC4_3.5x3.5mm_P1.75mm, symbol LED:SK6812MINI
- added D66: PgUpRGB, LED_SMD:LED_SK6812MINI_PLCC4_3.5x3.5mm_P1.75mm, symbol LED:SK6812MINI
- added D83: TabRGB, LED_SMD:LED_SK6812MINI_PLCC4_3.5x3.5mm_P1.75mm, symbol LED:SK6812MINI
- added D84: QRGB, LED_SMD:LED_SK6812MINI_PLCC4_3.5x3.5mm_P1.75mm, symbol LED:SK6812MINI
- added D85: WRGB, LED_SMD:LED_SK6812MINI_PLCC4_3.5x3.5mm_P1.75mm, symbol LED:SK6812MINI
- added D86: ERGB, LED_SMD:LED_SK6812MINI_PLCC4_3.5x3.5mm_P1.75mm, symbol LED:SK6812MINI
- added D87: RRGB, LED_SMD:LED_SK6812MINI_PLCC4_3.5x3.5mm_P1.75mm, symbol LED:SK6812MINI
- added D88: TRGB, LED_SMD:LED_SK6812MINI_PLCC4_3.5x3.5mm_P1.75mm, symbol LED:SK6812MINI
- added D89: YRGB, LED_SMD:LED_SK6812MINI_PLCC4_3.5x3.5mm_P1.75mm, symbol LED:SK6812MINI
- added D90: URGB, LED_SMD:LED_SK6812MINI_PLCC4_3.5x3.5mm_P1.75mm, symbol LED:SK6812MINI
- added D91: IRGB, LED_SMD:LED_SK6812MINI_PLCC4_3.5x3.5mm_P1.75mm, symbol LED:SK6812MINI
- added D92: ORGB, LED_SMD:LED_SK6812MINI_PLCC4_3.5x3.5mm_P1.75mm, symbol LED:SK6812MINI
- added D93: PRGB, LED_SMD:LED_SK6812MINI_PLCC4_3.5x3.5mm_P1.75mm, symbol LED:SK6812MINI
- added D94: [RGB, LED_SMD:LED_SK6812MINI_PLCC4_3.5x3.5mm_P1.75mm, symbol LED:SK6812MINI
- added D95: ]RGB, LED_SMD:LED_SK6812MINI_PLCC4_3.5x3.5mm_P1.75mm, symbol LED:SK6812MINI
- added D96: EnterRGB, LED_SMD:LED_SK6812MINI_PLCC4_3.5x3.5mm_P1.75mm, symbol LED:SK6812MINI
- added D97: DeleteRGB, LED_SMD:LED_SK6812MINI_PLCC4_3.5x3.5mm_P1.75mm, symbol LED:SK6812MINI
- added D98: PgDnRGB, LED_SMD:LED_SK6812MINI_PLCC4_3.5x3.5mm_P1.75mm, symbol LED:SK6812MINI
- SW1: value ESC -> SW_Push
- SW2: value F1 -> SW_Push
- SW3: value F2 -> SW_Push
Connections:
- net row3 is gone; now on an unnamed net: D50.1 (K)
- net row5 is gone; now on an unnamed net: D81.1 (K), D82.1 (K)
- net at SW36.1: now also D69.2 (A); no longer D36.2 (A)
- net at SW57.1: now also D106.2 (A)
- net at SW87.1: now also D167.2 (A)
- net at SW26.1: now also D43.2 (A)
- net at SW43.1: now also D76.2 (A); no longer D43.2 (A)
- net at SW38.1: now also D71.2 (A); no longer D38.2 (A)
- net at SW35.1: now also D68.2 (A); no longer D35.2 (A)
- net at SW25.1: now also D42.2 (A)
- net at SW63.1: now also D112.2 (A)
- net at SW65.1: now also D129.2 (A)
- net at SW22.1: now also D39.2 (A)
- net at SW64.1: now also D113.2 (A)
- net at SW90.1: now also D170.2 (A)
- net at SW34.1: now also D67.2 (A)
- net at SW41.1: now also D74.2 (A); no longer D41.2 (A)
- net at SW69.1: now also D133.2 (A); no longer D69.2 (A)
- net at SW24.1: now also D41.2 (A)
- net at SW60.1: now also D109.2 (A)
- net at SW53.1: now also D102.2 (A)
- net at SW84.1: now also D164.2 (A)
- net at SW88.1: now also D168.2 (A)
- net at SW81.1: now also D161.2 (A); no longer D81.2 (A)
- net at SW67.1: now also D131.2 (A); no longer D67.2 (A)
- net at SW42.1: now also D75.2 (A); no longer D42.2 (A)
- net at SW27.1: now also D44.2 (A)
- net at SW61.1: now also D110.2 (A)
- net at SW19.1: now also D36.2 (A)
- net at SW76.1: now also D140.2 (A); no longer D76.2 (A)
- net at SW51.1: now also D100.2 (A)
- net at SW32.1: now also D49.2 (A)
- net at SW62.1: now also D111.2 (A)
- net at SW58.1: now also D107.2 (A)
- net at SW50.1: now also D99.2 (A); no longer D50.2 (A)
- net at SW23.1: now also D40.2 (A)
- net at SW28.1: now also D45.2 (A)
- net at SW49.1: now also D82.2 (A); no longer D49.2 (A)
- net at SW85.1: now also D165.2 (A)
- net at SW83.1: now also D163.2 (A)
- net at SW75.1: now also D139.2 (A); no longer D75.2 (A)
- net at SW20.1: now also D37.2 (A)
- net at SW89.1: now also D169.2 (A)
- net at D80.2 (A): now also SW47.1; no longer SW80.1
- net at SW91.1: now also D171.2 (A)
- net at SW30.1: now also D47.2 (A)
- net at SW66.1: now also D130.2 (A)
- net at D72.2 (A): now also SW39.1; no longer SW72.1
- net at SW31.1: now also D48.2 (A)
- net at SW33.1: now also D50.2 (A)
- net at SW82.1: now also D162.2 (A); no longer D82.2 (A)
- net at SW59.1: now also D108.2 (A)
- net at SW71.1: now also D135.2 (A); no longer D71.2 (A)
- net at SW54.1: now also D103.2 (A)
- net at SW73.1: now also D137.2 (A); no longer D73.2 (A)
- net at SW44.1: now also D77.2 (A); no longer D44.2 (A)
- net at SW45.1: now also D78.2 (A); no longer D45.2 (A)
- net at D46.2 (A): now also SW29.1; no longer SW46.1
- net at SW56.1: now also D105.2 (A)
- net at SW78.1: now also D142.2 (A); no longer D78.2 (A)
- net at SW52.1: now also D101.2 (A)
- net at SW68.1: now also D132.2 (A); no longer D68.2 (A)
- net at SW74.1: now also D138.2 (A); no longer D74.2 (A)
- net at SW21.1: now also D38.2 (A)
- net at SW86.1: now also D166.2 (A)
- net at SW77.1: now also D141.2 (A); no longer D77.2 (A)
- net at SW18.1: now also D35.2 (A)
- net at SW70.1: now also D134.2 (A); no longer D70.2 (A)
- net at SW48.1: now also D81.2 (A); no longer D48.2 (A)
- net at SW79.1: now also D143.2 (A); no longer D79.2 (A)
- net at SW37.1: now also D70.2 (A); no longer D37.2 (A)
- net at SW40.1: now also D73.2 (A); no longer D40.2 (A)
- net at SW55.1: now also D104.2 (A)
- net col0: no longer names the net of SW1.2, SW18.2, SW34.2, SW50.2, SW65.2, SW81.2
- net col1: no longer names the net of SW19.2, SW2.2, SW35.2, SW51.2, SW66.2, SW82.2
- net col10: no longer names the net of SW11.2, SW28.2, SW44.2, SW60.2, SW75.2, SW85.2
- net col11: no longer names the net of SW12.2, SW29.2, SW45.2, SW61.2, SW76.2, SW86.2
- net col12: no longer names the net of SW13.2, SW30.2, SW46.2, SW62.2, SW77.2, SW87.2
- net col13: no longer names the net of SW14.2, SW31.2, SW47.2, SW78.2, SW88.2
- net col13: no longer SW63.2
- net col14: no longer names the net of SW15.2, SW89.2
- net col14: no longer SW48.2
- net col15: no longer names the net of SW16.2, SW32.2, SW79.2, SW90.2
- net col15: now also SW48.2, SW63.2
- net col16: no longer names the net of SW17.2, SW33.2, SW49.2, SW64.2, SW80.2, SW91.2
- net col2: no longer names the net of SW20.2, SW3.2, SW36.2, SW52.2, SW67.2, SW83.2
- net col3: no longer names the net of SW21.2, SW37.2, SW4.2, SW53.2, SW68.2
- net col4: no longer names the net of SW22.2, SW38.2, SW5.2, SW54.2, SW69.2
- net col5: no longer names the net of SW23.2, SW39.2, SW55.2, SW6.2, SW70.2
- net col6: no longer names the net of SW24.2, SW40.2, SW56.2, SW7.2, SW71.2, SW84.2
- net col7: no longer names the net of SW25.2, SW41.2, SW57.2, SW72.2, SW8.2
- net col8: no longer names the net of SW26.2, SW42.2, SW58.2, SW73.2, SW9.2
- net col9: no longer names the net of SW10.2, SW27.2, SW43.2, SW59.2, SW74.2
- net row0: no longer names the net of D1.1 (K), D10.1 (K), D11.1 (K), D12.1 (K), D13.1 (K), D14.1 (K), D15.1 (K), D16.1 (K), D17.1 (K), D2.1 (K), D3.1 (K), D4.1 (K), D5.1 (K), D6.1 (K), D7.1 (K), D8.1 (K), D9.1 (K)
- net row2: no longer names the net of D35.1 (K), D36.1 (K), D37.1 (K), D38.1 (K), D39.1 (K), D40.1 (K), D41.1 (K), D42.1 (K), D43.1 (K), D44.1 (K), D45.1 (K), D46.1 (K), D47.1 (K), D48.1 (K), D49.1 (K)
- net row4: no longer names the net of D67.1 (K), D68.1 (K), D69.1 (K), D70.1 (K), D71.1 (K), D72.1 (K), D73.1 (K), D74.1 (K), D75.1 (K), D76.1 (K), D77.1 (K), D78.1 (K), D79.1 (K), D80.1 (K)
- new net: D173.1 (DOUT), D174.3 (DIN)
- new net: D172.1 (DOUT), D173.3 (DIN)
- new net: D129.1 (K), D130.1 (K), D131.1 (K), D132.1 (K), D133.1 (K), D134.1 (K), D135.1 (K), D136.1 (K), D137.1 (K), D138.1 (K), D139.1 (K), D140.1 (K), D141.1 (K), D142.1 (K), D143.1 (K), D144.1 (K)
- new net: D100.1 (K), D101.1 (K), D102.1 (K), D103.1 (K), D104.1 (K), D105.1 (K), D106.1 (K), D107.1 (K), D108.1 (K), D109.1 (K), D110.1 (K), D111.1 (K), D112.1 (K), D113.1 (K), D99.1 (K)
- new net: D114.3 (DIN), D98.1 (DOUT)
- new net: D97.1 (DOUT), D98.3 (DIN)
- new net: D20.1 (DOUT), D21.3 (DIN)
- new net: D19.1 (DOUT), D20.3 (DIN)
- new net: D127.1 (DOUT), D128.3 (DIN)
- new net: D126.1 (DOUT), D127.3 (DIN)
- new net: D145.1 (DOUT), D146.3 (DIN)
- new net: D128.1 (DOUT), D145.3 (DIN)
- new net: D144.2 (A), SW80.1
- new net: D63.1 (DOUT), D64.3 (DIN)
- new net: D62.1 (DOUT), D63.3 (DIN)
- new net: D161.1 (K), D162.1 (K), D163.1 (K), D164.1 (K), D165.1 (K), D166.1 (K), D167.1 (K), D168.1 (K), D169.1 (K), D170.1 (K), D171.1 (K)
- new net: D159.1 (DOUT), D160.3 (DIN)
- new net: D158.1 (DOUT), D159.3 (DIN)
- new net: D59.1 (DOUT), D60.3 (DIN)
- new net: D58.1 (DOUT), D59.3 (DIN)
- new net: D57.1 (DOUT), D58.3 (DIN)
- new net: D61.1 (DOUT), D62.3 (DIN)
- new net: D60.1 (DOUT), D61.3 (DIN)
- new net: D146.1 (DOUT), D147.3 (DIN)
- new net: D179.1 (DOUT), D180.3 (DIN)
- new net: D178.1 (DOUT), D179.3 (DIN)
- new net: D122.1 (DOUT), D123.3 (DIN)
- new net: D121.1 (DOUT), D122.3 (DIN)
- new net: D154.1 (DOUT), D155.3 (DIN)
- new net: D153.1 (DOUT), D154.3 (DIN)
- new net: D92.1 (DOUT), D93.3 (DIN)
- new net: D91.1 (DOUT), D92.3 (DIN)
- new net: D160.1 (DOUT), D172.3 (DIN)
- new net: D90.1 (DOUT), D91.3 (DIN)
- new net: D180.1 (DOUT), D181.3 (DIN)
- new net: D64.1 (DOUT), D65.3 (DIN)
- new net: D123.1 (DOUT), D124.3 (DIN)
- new net: D124.1 (DOUT), D125.3 (DIN)
- new net: D136.2 (A), SW72.1
- new net: D22.1 (DOUT), D23.3 (DIN)
- new net: D21.1 (DOUT), D22.3 (DIN)
- new net: D23.1 (DOUT), D24.3 (DIN)
- new net: D79.2 (A), SW46.1
- new net: D84.1 (DOUT), D85.3 (DIN)
- new net: D83.1 (DOUT), D84.3 (DIN)
- new net: D120.1 (DOUT), D121.3 (DIN)
- new net: D119.1 (DOUT), D120.3 (DIN)
- new net: D96.1 (DOUT), D97.3 (DIN)
- new net: D95.1 (DOUT), D96.3 (DIN)
- new net: D149.1 (DOUT), D150.3 (DIN)
- new net: D148.1 (DOUT), D149.3 (DIN)
- new net: D66.1 (DOUT), D83.3 (DIN)
- new net: D65.1 (DOUT), D66.3 (DIN)
- new net: D51.1 (DOUT), D52.3 (DIN)
- new net: D34.1 (DOUT), D51.3 (DIN)
- new net: D88.1 (DOUT), D89.3 (DIN)
- new net: D87.1 (DOUT), D88.3 (DIN)
- new net: D93.1 (DOUT), D94.3 (DIN)
- new net: D94.1 (DOUT), D95.3 (DIN)
- new net: D56.1 (DOUT), D57.3 (DIN)
- new net: D55.1 (DOUT), D56.3 (DIN)
- new net: D18.1 (DOUT), D19.3 (DIN)
- new net: D86.1 (DOUT), D87.3 (DIN)
- new net: D85.1 (DOUT), D86.3 (DIN)
- new net: D147.1 (DOUT), D148.3 (DIN)
- new net: D152.1 (DOUT), D153.3 (DIN)
- new net: D31.1 (DOUT), D32.3 (DIN)
- new net: D30.1 (DOUT), D31.3 (DIN)
- new net: D118.1 (DOUT), D119.3 (DIN)
- new net: D117.1 (DOUT), D118.3 (DIN)
- new net: D157.1 (DOUT), D158.3 (DIN)
- new net: D156.1 (DOUT), D157.3 (DIN)
- new net: D181.1 (DOUT), D182.3 (DIN)
- new net: D125.1 (DOUT), D126.3 (DIN)
- new net: D33.1 (DOUT), D34.3 (DIN)
- new net: D26.1 (DOUT), D27.3 (DIN)
- new net: D25.1 (DOUT), D26.3 (DIN)
- new net: D151.1 (DOUT), D152.3 (DIN)
- new net: D177.1 (DOUT), D178.3 (DIN)
- new net: D176.1 (DOUT), D177.3 (DIN)
- new net: D54.1 (DOUT), D55.3 (DIN)
- new net: D53.1 (DOUT), D54.3 (DIN)
- new net: D150.1 (DOUT), D151.3 (DIN)
- new net: D175.1 (DOUT), D176.3 (DIN)
- new net: D24.1 (DOUT), D25.3 (DIN)
- new net: D29.1 (DOUT), D30.3 (DIN)
- new net: D27.1 (DOUT), D28.3 (DIN)
- new net: D116.1 (DOUT), D117.3 (DIN)
- new net: D115.1 (DOUT), D116.3 (DIN)
- new net: D52.1 (DOUT), D53.3 (DIN)
- new net: D28.1 (DOUT), D29.3 (DIN)
- new net: D32.1 (DOUT), D33.3 (DIN)
- new net: D155.1 (DOUT), D156.3 (DIN)
- new net: D89.1 (DOUT), D90.3 (DIN)
- new net: D174.1 (DOUT), D175.3 (DIN)
- new net: D114.1 (DOUT), D115.3 (DIN)
- new net GND: D114.2 (VSS), D115.2 (VSS), D116.2 (VSS), D117.2 (VSS), D118.2 (VSS), D119.2 (VSS), D120.2 (VSS), D121.2 (VSS), D122.2 (VSS), D123.2 (VSS), D124.2 (VSS), D125.2 (VSS), D126.2 (VSS), D127.2 (VSS), D128.2 (VSS), D145.2 (VSS), D146.2 (VSS), D147.2 (VSS), D148.2 (VSS), D149.2 (VSS), D150.2 (VSS), D151.2 (VSS), D152.2 (VSS), D153.2 (VSS), D154.2 (VSS), D155.2 (VSS), D156.2 (VSS), D157.2 (VSS), D158.2 (VSS), D159.2 (VSS), D160.2 (VSS), D172.2 (VSS), D173.2 (VSS), D174.2 (VSS), D175.2 (VSS), D176.2 (VSS), D177.2 (VSS), D178.2 (VSS), D179.2 (VSS), D18.2 (VSS), D180.2 (VSS), D181.2 (VSS), D182.2 (VSS), D19.2 (VSS), D20.2 (VSS), D21.2 (VSS), D22.2 (VSS), D23.2 (VSS), D24.2 (VSS), D25.2 (VSS), D26.2 (VSS), D27.2 (VSS), D28.2 (VSS), D29.2 (VSS), D30.2 (VSS), D31.2 (VSS), D32.2 (VSS), D33.2 (VSS), D34.2 (VSS), D51.2 (VSS), D52.2 (VSS), D53.2 (VSS), D54.2 (VSS), D55.2 (VSS), D56.2 (VSS), D57.2 (VSS), D58.2 (VSS), D59.2 (VSS), D60.2 (VSS), D61.2 (VSS), D62.2 (VSS), D63.2 (VSS), D64.2 (VSS), D65.2 (VSS), D66.2 (VSS), D83.2 (VSS), D84.2 (VSS), D85.2 (VSS), D86.2 (VSS), D87.2 (VSS), D88.2 (VSS), D89.2 (VSS), D90.2 (VSS), D91.2 (VSS), D92.2 (VSS), D93.2 (VSS), D94.2 (VSS), D95.2 (VSS), D96.2 (VSS), D97.2 (VSS), D98.2 (VSS)
- new net VCC: D114.4 (VDD), D115.4 (VDD), D116.4 (VDD), D117.4 (VDD), D118.4 (VDD), D119.4 (VDD), D120.4 (VDD), D121.4 (VDD), D122.4 (VDD), D123.4 (VDD), D124.4 (VDD), D125.4 (VDD), D126.4 (VDD), D127.4 (VDD), D128.4 (VDD), D145.4 (VDD), D146.4 (VDD), D147.4 (VDD), D148.4 (VDD), D149.4 (VDD), D150.4 (VDD), D151.4 (VDD), D152.4 (VDD), D153.4 (VDD), D154.4 (VDD), D155.4 (VDD), D156.4 (VDD), D157.4 (VDD), D158.4 (VDD), D159.4 (VDD), D160.4 (VDD), D172.4 (VDD), D173.4 (VDD), D174.4 (VDD), D175.4 (VDD), D176.4 (VDD), D177.4 (VDD), D178.4 (VDD), D179.4 (VDD), D18.4 (VDD), D180.4 (VDD), D181.4 (VDD), D182.4 (VDD), D19.4 (VDD), D20.4 (VDD), D21.4 (VDD), D22.4 (VDD), D23.4 (VDD), D24.4 (VDD), D25.4 (VDD), D26.4 (VDD), D27.4 (VDD), D28.4 (VDD), D29.4 (VDD), D30.4 (VDD), D31.4 (VDD), D32.4 (VDD), D33.4 (VDD), D34.4 (VDD), D51.4 (VDD), D52.4 (VDD), D53.4 (VDD), D54.4 (VDD), D55.4 (VDD), D56.4 (VDD), D57.4 (VDD), D58.4 (VDD), D59.4 (VDD), D60.4 (VDD), D61.4 (VDD), D62.4 (VDD), D63.4 (VDD), D64.4 (VDD), D65.4 (VDD), D66.4 (VDD), D83.4 (VDD), D84.4 (VDD), D85.4 (VDD), D86.4 (VDD), D87.4 (VDD), D88.4 (VDD), D89.4 (VDD), D90.4 (VDD), D91.4 (VDD), D92.4 (VDD), D93.4 (VDD), D94.4 (VDD), D95.4 (VDD), D96.4 (VDD), D97.4 (VDD), D98.4 (VDD)

Commit message: v1xa
Parts:
- SW1: value SW_Push -> ESC
- SW10: value SW_Push -> F8
- SW11: value SW_Push -> F9
- SW12: value SW_Push -> F10
- SW13: value SW_Push -> F11
- SW14: value SW_Push -> F12
- SW15: value SW_Push -> U1
- SW16: value SW_Push -> PrtSc
- SW17: value SW_Push -> PauseBr
- SW18: value SW_Push -> `
- SW19: value SW_Push -> #1
- SW2: value SW_Push -> F1
- SW20: value SW_Push -> #2
- SW21: value SW_Push -> #3
- SW22: value SW_Push -> #4
- SW23: value SW_Push -> #5
- SW24: value SW_Push -> #6
- SW25: value SW_Push -> #7
- SW26: value SW_Push -> #8
- SW27: value SW_Push -> #9
- SW28: value SW_Push -> #0
- SW29: value SW_Push -> -
- SW3: value SW_Push -> F2
- SW30: value SW_Push -> =
- SW31: value SW_Push -> BackSpace
- SW32: value SW_Push -> Insert
- SW33: value SW_Push -> PgUp
- SW34: value SW_Push -> Tab
- SW35: value SW_Push -> Q
- SW36: value SW_Push -> W
- SW37: value SW_Push -> E
- SW38: value SW_Push -> R
- SW39: value SW_Push -> T
- SW4: value SW_Push -> F3
- SW40: value SW_Push -> Y
- SW41: value SW_Push -> U
- SW42: value SW_Push -> I
- SW43: value SW_Push -> O
- SW44: value SW_Push -> P
- SW45: value SW_Push -> [
- SW46: value SW_Push -> ]
- SW47: value SW_Push -> Enter
- SW48: value SW_Push -> Delete
- SW49: value SW_Push -> PgDn
- SW5: value SW_Push -> F4
- SW50: value SW_Push -> CapsLock
- SW51: value SW_Push -> A
- SW52: value SW_Push -> S
- SW53: value SW_Push -> D
- SW54: value SW_Push -> F
- SW55: value SW_Push -> G
- SW56: value SW_Push -> H
- SW57: value SW_Push -> J
- SW58: value SW_Push -> K
- SW59: value SW_Push -> L
- SW6: value SW_Push -> F5
- SW60: value SW_Push -> ;
- SW61: value SW_Push -> '@
- SW62: value SW_Push -> #~
- SW63: value SW_Push -> Home
- SW64: value SW_Push -> End
- SW65: value SW_Push -> LShift
- SW66: value SW_Push -> \|
- SW67: value SW_Push -> Z
- SW68: value SW_Push -> X
- SW69: value SW_Push -> C
- SW7: value SW_Push -> F6
- SW70: value SW_Push -> V
- SW71: value SW_Push -> B
- SW72: value SW_Push -> N
- SW73: value SW_Push -> M
- SW74: value SW_Push -> ,<
- SW75: value SW_Push -> .>
- SW76: value SW_Push -> /?
- SW77: value SW_Push -> RShift
- SW78: value SW_Push -> UpArrow
- SW79: value SW_Push -> U2
- SW8: value SW_Push -> XEV
- SW80: value SW_Push -> U3
- SW81: value SW_Push -> LCtrl
- SW82: value SW_Push -> Win
- SW83: value SW_Push -> Alt
- SW84: value SW_Push -> Space
- SW85: value SW_Push -> AltGr
- SW86: value SW_Push -> Fn
- SW87: value SW_Push -> RCtrl
- SW88: value SW_Push -> LeftArrow
- SW89: value SW_Push -> DownArrow
- SW9: value SW_Push -> F7
- SW90: value SW_Push -> RightArrow
- SW91: value SW_Push -> U4
Connections:
- net col8: now reaches SW26.2, SW42.2, SW58.2, SW73.2, SW9.2
- net row4: now reaches D129.1 (K), D130.1 (K), D131.1 (K), D132.1 (K), D133.1 (K), D134.1 (K), D135.1 (K), D136.1 (K), D137.1 (K), D138.1 (K), D139.1 (K), D140.1 (K), D141.1 (K), D142.1 (K), D143.1 (K), D144.1 (K)
- net col15: now reaches SW16.2, SW32.2, SW48.2, SW63.2, SW79.2, SW90.2
- net row3: now reaches D100.1 (K), D101.1 (K), D102.1 (K), D103.1 (K), D104.1 (K), D105.1 (K), D106.1 (K), D107.1 (K), D108.1 (K), D109.1 (K), D110.1 (K), D111.1 (K), D112.1 (K), D113.1 (K), D99.1 (K)
- net row1: now reaches D35.1 (K), D36.1 (K), D37.1 (K), D38.1 (K), D39.1 (K), D40.1 (K), D41.1 (K), D42.1 (K), D43.1 (K), D44.1 (K), D45.1 (K), D46.1 (K), D47.1 (K), D48.1 (K), D49.1 (K), D50.1 (K)
- net row2: now reaches D67.1 (K), D68.1 (K), D69.1 (K), D70.1 (K), D71.1 (K), D72.1 (K), D73.1 (K), D74.1 (K), D75.1 (K), D76.1 (K), D77.1 (K), D78.1 (K), D79.1 (K), D80.1 (K), D81.1 (K), D82.1 (K)
- net col6: now reaches SW24.2, SW40.2, SW56.2, SW7.2, SW71.2, SW84.2
- net col12: now reaches SW13.2, SW30.2, SW46.2, SW62.2, SW77.2, SW87.2
- net col16: now reaches SW17.2, SW33.2, SW49.2, SW64.2, SW80.2, SW91.2
- net col10: now reaches SW11.2, SW28.2, SW44.2, SW60.2, SW75.2, SW85.2
- net col9: now reaches SW10.2, SW27.2, SW43.2, SW59.2, SW74.2
- net row5: now reaches D161.1 (K), D162.1 (K), D163.1 (K), D164.1 (K), D165.1 (K), D166.1 (K), D167.1 (K), D168.1 (K), D169.1 (K), D170.1 (K), D171.1 (K)
- net col4: now reaches SW22.2, SW38.2, SW5.2, SW54.2, SW69.2
- net col5: now reaches SW23.2, SW39.2, SW55.2, SW6.2, SW70.2
- net col11: now reaches SW12.2, SW29.2, SW45.2, SW61.2, SW76.2, SW86.2
- net col1: now reaches SW19.2, SW2.2, SW35.2, SW51.2, SW66.2, SW82.2
- net row0: now reaches D1.1 (K), D10.1 (K), D11.1 (K), D12.1 (K), D13.1 (K), D14.1 (K), D15.1 (K), D16.1 (K), D17.1 (K), D2.1 (K), D3.1 (K), D4.1 (K), D5.1 (K), D6.1 (K), D7.1 (K), D8.1 (K), D9.1 (K)
- net col0: now reaches SW1.2, SW18.2, SW34.2, SW50.2, SW65.2, SW81.2
- net col13: now reaches SW14.2, SW31.2, SW47.2, SW78.2, SW88.2
- net col3: now reaches SW21.2, SW37.2, SW4.2, SW53.2, SW68.2
- net col2: now reaches SW20.2, SW3.2, SW36.2, SW52.2, SW67.2, SW83.2
- net led: now reaches D18.3 (DIN)
- net col7: now reaches SW25.2, SW41.2, SW57.2, SW72.2, SW8.2
- net col14: now reaches SW15.2, SW89.2

Commit message: v1za
Connections:
- no-connect marks 0 -> 1
Changed lines of the file:
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@@
   (junction (at 43.18 186.69) (diameter 0) (color 0 0 0 0)
   )
+  (junction (at 490.22 153.67) (diameter 0) (color 0 0 0 0)
+  )
   (junction (at 123.19 186.69) (diameter 0) (color 0 0 0 0)
   )
@@
   (junction (at 469.9 256.54) (diameter 0) (color 0 0 0 0)
   )
-  (junction (at 283.21 153.67) (diameter 0) (color 0 0 0 0)
-  )
   (junction (at 69.85 340.36) (diameter 0) (color 0 0 0 0)
   )
@@
   (junction (at 176.53 289.56) (diameter 0) (color 0 0 0 0)
   )
+  (junction (at 283.21 153.67) (diameter 0) (color 0 0 0 0)
+  )
   (junction (at 443.23 152.4) (diameter 0) (color 0 0 0 0)
   )
@@
   (junction (at 469.9 222.25) (diameter 0) (color 0 0 0 0)
   )
+  (no_connect (at 477.52 332.74))
   (wire (pts (xy 363.22 187.96) (xy 389.89 187.96))
     (stroke (width 0) (type default) (color 0 0 0 0))
@@
     (stroke (width 0) (type default) (color 0 0 0 0))
   )
-  (wire (pts (xy 469.9 153.67) (xy 496.57 153.67))
+  (wire (pts (xy 469.9 153.67) (xy 490.22 153.67))
     (stroke (width 0) (type default) (color 0 0 0 0))
   )
@@
     (stroke (width 0) (type default) (color 0 0 0 0))
   )
+  (wire (pts (xy 490.22 160.02) (xy 490.22 153.67))
+    (stroke (width 0) (type default) (color 0 0 0 0))
+  )
   (wire (pts (xy 290.83 298.45) (xy 302.26 298.45))
     (stroke (width 0) (type default) (color 0 0 0 0))
@@
     (stroke (width 0) (type default) (color 0 0 0 0))
   )
+  (wire (pts (xy 497.84 160.02) (xy 490.22 160.02))
+    (stroke (width 0) (type default) (color 0 0 0 0))
+  )
   (wire (pts (xy 157.48 161.29) (xy 168.91 161.29))
     (stroke (width 0) (type default) (color 0 0 0 0))
@@
     (stroke (width 0) (type default) (color 0 0 0 0))
   )
-  (wire (pts (xy 283.21 153.67) (xy 309.88 153.67))
+  (wire (pts (xy 256.54 153.67) (xy 283.21 153.67))
     (stroke (width 0) (type default) (color 0 0 0 0))
   )
@@
     (stroke (width 0) (type default) (color 0 0 0 0))
   )
-  (wire (pts (xy 477.52 332.74) (xy 488.95 332.74))
-    (stroke (width 0) (type default) (color 0 0 0 0))
-  )
   (wire (pts (xy 373.38 318.77) (xy 373.38 353.06))
     (stroke (width 0) (type default) (color 0 0 0 0))
@@
     (stroke (width 0) (type default) (color 0 0 0 0))
   )
-  (wire (pts (xy 256.54 153.67) (xy 283.21 153.67))
-    (stroke (width 0) (type default) (color 0 0 0 0))
-  )
   (wire (pts (xy 469.9 152.4) (xy 496.57 152.4))
     (stroke (width 0) (type default) (color 0 0 0 0))
@@
     (stroke (width 0) (type default) (color 0 0 0 0))
   )
+  (wire (pts (xy 283.21 153.67) (xy 309.88 153.67))
+    (stroke (width 0) (type default) (color 0 0 0 0))
+  )
   (wire (pts (xy 416.56 168.91) (xy 443.23 168.91))
     (stroke (width 0) (type default) (color 0 0 0 0))
@@
     (stroke (width 0) (type default) (color 0 0 0 0))
   )
+  (wire (pts (xy 490.22 153.67) (xy 496.57 153.67))
+    (stroke (width 0) (type default) (color 0 0 0 0))
+  )
   (wire (pts (xy 443.23 168.91) (xy 469.9 168.91))
     (stroke (width 0) (type default) (color 0 0 0 0))
@@
     (pin "4")
   )
+  (symbol (lib_id "power:PWR_FLAG") (at 497.84 160.02 0) (unit 1)
+    (in_bom yes) (on_board yes) (fields_autoplaced)
+    (property "Reference" "#FLG02" (id 0) (at 497.84 158.115 0)
+      (effects (font (size 1.27 1.27)) hide)
+    )
+    (property "Value" "PWR_FLAG" (id 1) (at 497.84 154.94 0))
+    (property "Footprint" "" (id 2) (at 497.84 160.02 0)
+      (effects (font (size 1.27 1.27)) hide)
+    )
+    (property "Datasheet" "~" (id 3) (at 497.84 160.02 0)
+      (effects (font (size 1.27 1.27)) hide)
+    )
+    (pin "1")
+  )
   (symbol (lib_id "Switch:SW_Push") (at 101.6 215.9 0) (unit 1)
