File: X95X/untitled.kicad_sch (KiCad schematic)
At the start: 273 parts, among them SW1 ESC, SW10 F8, SW11 F9, SW12 F10, SW13 F11, SW14 F12, SW15 U1, SW16 PrtSc, SW17 PauseBr, SW18 `, SW19 #1, SW2 F1, SW20 #2, SW21 #3, SW22 #4, SW23 #5, SW24 #6, SW25 #7, SW26 #8, SW27 #9, SW28 #0, SW29 -, SW3 F2, SW30 =, SW31 BackSpace, SW32 Insert, SW33 PgUp, SW34 Tab, SW35 Q, SW36 W, SW37 E, SW38 R, SW39 T, SW4 F3, SW40 Y, SW41 U, SW42 I, SW43 O, SW44 P, SW45 [, SW46 ], SW47 Enter, SW48 Delete, SW49 PgDn, SW5 F4, SW50 CapsLock, SW51 A, SW52 S, SW53 D, SW54 F, SW55 G, SW56 H, SW57 J, SW58 K, SW59 L, SW6 F5, SW60 ;, SW61 '@, SW62 #~, SW63 Home, SW64 End, SW65 LShift, SW66 \|, SW67 Z, SW68 X, SW69 C, SW7 F6, SW70 V, SW71 B, SW72 N, SW73 M, SW74 ,<, SW75 .>, SW76 /?, SW77 RShift, SW78 UpArrow, SW79 U2, SW8 XEV, SW80 U3, SW81 LCtrl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

Commit message: PCB!!!
Parts:
- SW1, SW10, SW11, SW12, SW13, SW14, SW15, SW16, SW17, SW18, SW19, SW2, SW20, SW21, SW22, SW23, SW24, SW25, SW26, SW27, SW28, SW29, SW3, SW30, SW31, SW32, SW33, SW35, SW36, SW37, SW38, SW39, SW4, SW40, SW41, SW42, SW43, SW44, SW45, SW46, SW47, SW48, SW49, SW5, SW51, SW52, SW53, SW54, SW55, SW56, SW57, SW58, SW59, SW6, SW60, SW61, SW62, SW63, SW64, SW66, SW67, SW68, SW69, SW7, SW70, SW71, SW72, SW73, SW74, SW75, SW76, SW78, SW79, SW8, SW80, SW84, SW85, SW86, SW87, SW88, SW89, SW9, SW90, SW91: footprint (none) -> marbastlib-mx:SW_MX_1u
- SW34: footprint (none) -> marbastlib-mx:SW_MX_1.5u
- SW50, SW77: footprint (none) -> marbastlib-mx:SW_MX_1.75u
- SW65, SW81, SW82, SW83: footprint (none) -> marbastlib-mx:SW_MX_1.25u

Commit message: more pcb
Parts:
- removed D100, D101, D102, D103, D104, D105, D106, D107, D108, D109, D110, D111, D112, D113, D129, D130, D131, D132, D133, D134, D135, D136, D137, D138, D139, D140, D141, D142, D143, D144, D161, D162, D163, D164, D165, D166, D167, D168, D169, D170, D171, D99: D_Small, Diode_SMD:D_SOD-123, symbol Device:D_Small
- removed D114: CapsLockRGB, LED_SMD:LED_SK6812MINI_PLCC4_3.5x3.5mm_P1.75mm, symbol LED:SK6812MINI
- removed D115: ARGB, LED_SMD:LED_SK6812MINI_PLCC4_3.5x3.5mm_P1.75mm, symbol LED:SK6812MINI
- removed D116: SRGB, LED_SMD:LED_SK6812MINI_PLCC4_3.5x3.5mm_P1.75mm, symbol LED:SK6812MINI
- removed D117: DRGB, LED_SMD:LED_SK6812MINI_PLCC4_3.5x3.5mm_P1.75mm, symbol LED:SK6812MINI
- removed D118: FRGB, LED_SMD:LED_SK6812MINI_PLCC4_3.5x3.5mm_P1.75mm, symbol LED:SK6812MINI
- removed D119: GRGB, LED_SMD:LED_SK6812MINI_PLCC4_3.5x3.5mm_P1.75mm, symbol LED:SK6812MINI
- removed D120: HRGB, LED_SMD:LED_SK6812MINI_PLCC4_3.5x3.5mm_P1.75mm, symbol LED:SK6812MINI
- removed D121: JRGB, LED_SMD:LED_SK6812MINI_PLCC4_3.5x3.5mm_P1.75mm, symbol LED:SK6812MINI
- removed D122: KRGB, LED_SMD:LED_SK6812MINI_PLCC4_3.5x3.5mm_P1.75mm, symbol LED:SK6812MINI
- removed D123: LRGB, LED_SMD:LED_SK6812MINI_PLCC4_3.5x3.5mm_P1.75mm, symbol LED:SK6812MINI
- removed D124: ;RGB, LED_SMD:LED_SK6812MINI_PLCC4_3.5x3.5mm_P1.75mm, symbol LED:SK6812MINI
- removed D125: '@RGB, LED_SMD:LED_SK6812MINI_PLCC4_3.5x3.5mm_P1.75mm, symbol LED:SK6812MINI
- removed D126: #~RGB, LED_SMD:LED_SK6812MINI_PLCC4_3.5x3.5mm_P1.75mm, symbol LED:SK6812MINI
- removed D127: HomeRGB, LED_SMD:LED_SK6812MINI_PLCC4_3.5x3.5mm_P1.75mm, symbol LED:SK6812MINI
- removed D128: EndRGB, LED_SMD:LED_SK6812MINI_PLCC4_3.5x3.5mm_P1.75mm, symbol LED:SK6812MINI
- removed D145: LShift, LED_SMD:LED_SK6812MINI_PLCC4_3.5x3.5mm_P1.75mm, symbol LED:SK6812MINI
- removed D146: \|RGB, LED_SMD:LED_SK6812MINI_PLCC4_3.5x3.5mm_P1.75mm, symbol LED:SK6812MINI
- removed D147: ZRGB, LED_SMD:LED_SK6812MINI_PLCC4_3.5x3.5mm_P1.75mm, symbol LED:SK6812MINI
- removed D148: XRGB, LED_SMD:LED_SK6812MINI_PLCC4_3.5x3.5mm_P1.75mm, symbol LED:SK6812MINI
- removed D149: CRGB, LED_SMD:LED_SK6812MINI_PLCC4_3.5x3.5mm_P1.75mm, symbol LED:SK6812MINI
- removed D150: VRGB, LED_SMD:LED_SK6812MINI_PLCC4_3.5x3.5mm_P1.75mm, symbol LED:SK6812MINI
- removed D151: BRGB, LED_SMD:LED_SK6812MINI_PLCC4_3.5x3.5mm_P1.75mm, symbol LED:SK6812MINI
- removed D152: NRGB, LED_SMD:LED_SK6812MINI_PLCC4_3.5x3.5mm_P1.75mm, symbol LED:SK6812MINI
- removed D153: MRGB, LED_SMD:LED_SK6812MINI_PLCC4_3.5x3.5mm_P1.75mm, symbol LED:SK6812MINI
- removed D154: ,<RGB, LED_SMD:LED_SK6812MINI_PLCC4_3.5x3.5mm_P1.75mm, symbol LED:SK6812MINI
- removed D155: .>RGB, LED_SMD:LED_SK6812MINI_PLCC4_3.5x3.5mm_P1.75mm, symbol LED:SK6812MINI
- removed D156: /?RGB, LED_SMD:LED_SK6812MINI_PLCC4_3.5x3.5mm_P1.75mm, symbol LED:SK6812MINI
- removed D157: RShiftRGB, LED_SMD:LED_SK6812MINI_PLCC4_3.5x3.5mm_P1.75mm, symbol LED:SK6812MINI
- removed D158: UpArrowRGB, LED_SMD:LED_SK6812MINI_PLCC4_3.5x3.5mm_P1.75mm, symbol LED:SK6812MINI
- removed D159: U2RGB, LED_SMD:LED_SK6812MINI_PLCC4_3.5x3.5mm_P1.75mm, symbol LED:SK6812MINI
- removed D160: U3RGB, LED_SMD:LED_SK6812MINI_PLCC4_3.5x3.5mm_P1.75mm, symbol LED:SK6812MINI
- removed D172: LCtrlRGB, LED_SMD:LED_SK6812MINI_PLCC4_3.5x3.5mm_P1.75mm, symbol LED:SK6812MINI
- removed D173: WinRGB, LED_SMD:LED_SK6812MINI_PLCC4_3.5x3.5mm_P1.75mm, symbol LED:SK6812MINI
- removed D174: AltRGB, LED_SMD:LED_SK6812MINI_PLCC4_3.5x3.5mm_P1.75mm, symbol LED:SK6812MINI
- removed D175: SpaceRGB, LED_SMD:LED_SK6812MINI_PLCC4_3.5x3.5mm_P1.75mm, symbol LED:SK6812MINI
- removed D176: AltGrRGB, LED_SMD:LED_SK6812MINI_PLCC4_3.5x3.5mm_P1.75mm, symbol LED:SK6812MINI
- removed D177: FnRGB, LED_SMD:LED_SK6812MINI_PLCC4_3.5x3.5mm_P1.75mm, symbol LED:SK6812MINI
- removed D178: RCtrlRGB, LED_SMD:LED_SK6812MINI_PLCC4_3.5x3.5mm_P1.75mm, symbol LED:SK6812MINI
- removed D179: LeftArrowRGB, LED_SMD:LED_SK6812MINI_PLCC4_3.5x3.5mm_P1.75mm, symbol LED:SK6812MINI
- removed D18: ESCRGB, LED_SMD:LED_SK6812MINI_PLCC4_3.5x3.5mm_P1.75mm, symbol LED:SK6812MINI
- removed D180: DownArrowRGB, LED_SMD:LED_SK6812MINI_PLCC4_3.5x3.5mm_P1.75mm, symbol LED:SK6812MINI
- removed D181: RightArrowRGB, LED_SMD:LED_SK6812MINI_PLCC4_3.5x3.5mm_P1.75mm, symbol LED:SK6812MINI
- removed D182: U4RGB, LED_SMD:LED_SK6812MINI_PLCC4_3.5x3.5mm_P1.75mm, symbol LED:SK6812MINI
- removed D19: F1RGB, LED_SMD:LED_SK6812MINI_PLCC4_3.5x3.5mm_P1.75mm, symbol LED:SK6812MINI
- removed D20: F2RGB, LED_SMD:LED_SK6812MINI_PLCC4_3.5x3.5mm_P1.75mm, symbol LED:SK6812MINI
- removed D21: F3RGB, LED_SMD:LED_SK6812MINI_PLCC4_3.5x3.5mm_P1.75mm, symbol LED:SK6812MINI
- removed D22: F4RGB, LED_SMD:LED_SK6812MINI_PLCC4_3.5x3.5mm_P1.75mm, symbol LED:SK6812MINI
- removed D23: F5RGB, LED_SMD:LED_SK6812MINI_PLCC4_3.5x3.5mm_P1.75mm, symbol LED:SK6812MINI
- removed D24: F6RGB, LED_SMD:LED_SK6812MINI_PLCC4_3.5x3.5mm_P1.75mm, symbol LED:SK6812MINI
- removed D25: XEVRGB, LED_SMD:LED_SK6812MINI_PLCC4_3.5x3.5mm_P1.75mm, symbol LED:SK6812MINI
- removed D26: F7RGB, LED_SMD:LED_SK6812MINI_PLCC4_3.5x3.5mm_P1.75mm, symbol LED:SK6812MINI
- removed D27: F8RGB, LED_SMD:LED_SK6812MINI_PLCC4_3.5x3.5mm_P1.75mm, symbol LED:SK6812MINI
- removed D28: F9RGB, LED_SMD:LED_SK6812MINI_PLCC4_3.5x3.5mm_P1.75mm, symbol LED:SK6812MINI
- removed D29: F10RGB, LED_SMD:LED_SK6812MINI_PLCC4_3.5x3.5mm_P1.75mm, symbol LED:SK6812MINI
- removed D30: F11RGB, LED_SMD:LED_SK6812MINI_PLCC4_3.5x3.5mm_P1.75mm, symbol LED:SK6812MINI
- removed D31: F12RGB, LED_SMD:LED_SK6812MINI_PLCC4_3.5x3.5mm_P1.75mm, symbol LED:SK6812MINI
- removed D32: U1RGB, LED_SMD:LED_SK6812MINI_PLCC4_3.5x3.5mm_P1.75mm, symbol LED:SK6812MINI
- removed D33: PrtScRGB, LED_SMD:LED_SK6812MINI_PLCC4_3.5x3.5mm_P1.75mm, symbol LED:SK6812MINI
- removed D34: PauseBrRGB, LED_SMD:LED_SK6812MINI_PLCC4_3.5x3.5mm_P1.75mm, symbol LED:SK6812MINI
- removed D51: `RGB, LED_SMD:LED_SK6812MINI_PLCC4_3.5x3.5mm_P1.75mm, symbol LED:SK6812MINI
- removed D52: 1RGB, LED_SMD:LED_SK6812MINI_PLCC4_3.5x3.5mm_P1.75mm, symbol LED:SK6812MINI
- removed D53: 2RGB, LED_SMD:LED_SK6812MINI_PLCC4_3.5x3.5mm_P1.75mm, symbol LED:SK6812MINI
- removed D54: 3RGB, LED_SMD:LED_SK6812MINI_PLCC4_3.5x3.5mm_P1.75mm, symbol LED:SK6812MINI
- removed D55: 4RGB, LED_SMD:LED_SK6812MINI_PLCC4_3.5x3.5mm_P1.75mm, symbol LED:SK6812MINI
- removed D56: 5RGB, LED_SMD:LED_SK6812MINI_PLCC4_3.5x3.5mm_P1.75mm, symbol LED:SK6812MINI
- removed D57: 6RGB, LED_SMD:LED_SK6812MINI_PLCC4_3.5x3.5mm_P1.75mm, symbol LED:SK6812MINI
- removed D58: 7RGB, LED_SMD:LED_SK6812MINI_PLCC4_3.5x3.5mm_P1.75mm, symbol LED:SK6812MINI
- removed D59: 8RGB, LED_SMD:LED_SK6812MINI_PLCC4_3.5x3.5mm_P1.75mm, symbol LED:SK6812MINI
- removed D60: 9RGB, LED_SMD:LED_SK6812MINI_PLCC4_3.5x3.5mm_P1.75mm, symbol LED:SK6812MINI
- removed D61: 0RGB, LED_SMD:LED_SK6812MINI_PLCC4_3.5x3.5mm_P1.75mm, symbol LED:SK6812MINI
- removed D62: -RGB, LED_SMD:LED_SK6812MINI_PLCC4_3.5x3.5mm_P1.75mm, symbol LED:SK6812MINI
- removed D63: =RGB, LED_SMD:LED_SK6812MINI_PLCC4_3.5x3.5mm_P1.75mm, symbol LED:SK6812MINI
- removed D64: BackSpaceRGB, LED_SMD:LED_SK6812MINI_PLCC4_3.5x3.5mm_P1.75mm, symbol LED:SK6812MINI
- removed D65: InsertRGB, LED_SMD:LED_SK6812MINI_PLCC4_3.5x3.5mm_P1.75mm, symbol LED:SK6812MINI
- removed D66: PgUpRGB, LED_SMD:LED_SK6812MINI_PLCC4_3.5x3.5mm_P1.75mm, symbol LED:SK6812MINI
- removed D83: TabRGB, LED_SMD:LED_SK6812MINI_PLCC4_3.5x3.5mm_P1.75mm, symbol LED:SK6812MINI
- removed D84: QRGB, LED_SMD:LED_SK6812MINI_PLCC4_3.5x3.5mm_P1.75mm, symbol LED:SK6812MINI
- removed D85: WRGB, LED_SMD:LED_SK6812MINI_PLCC4_3.5x3.5mm_P1.75mm, symbol LED:SK6812MINI
- removed D86: ERGB, LED_SMD:LED_SK6812MINI_PLCC4_3.5x3.5mm_P1.75mm, symbol LED:SK6812MINI
- removed D87: RRGB, LED_SMD:LED_SK6812MINI_PLCC4_3.5x3.5mm_P1.75mm, symbol LED:SK6812MINI
- removed D88: TRGB, LED_SMD:LED_SK6812MINI_PLCC4_3.5x3.5mm_P1.75mm, symbol LED:SK6812MINI
- removed D89: YRGB, LED_SMD:LED_SK6812MINI_PLCC4_3.5x3.5mm_P1.75mm, symbol LED:SK6812MINI
- removed D90: URGB, LED_SMD:LED_SK6812MINI_PLCC4_3.5x3.5mm_P1.75mm, symbol LED:SK6812MINI
- removed D91: IRGB, LED_SMD:LED_SK6812MINI_PLCC4_3.5x3.5mm_P1.75mm, symbol LED:SK6812MINI
- removed D92: ORGB, LED_SMD:LED_SK6812MINI_PLCC4_3.5x3.5mm_P1.75mm, symbol LED:SK6812MINI
- removed D93: PRGB, LED_SMD:LED_SK6812MINI_PLCC4_3.5x3.5mm_P1.75mm, symbol LED:SK6812MINI
- removed D94: [RGB, LED_SMD:LED_SK6812MINI_PLCC4_3.5x3.5mm_P1.75mm, symbol LED:SK6812MINI
- removed D95: ]RGB, LED_SMD:LED_SK6812MINI_PLCC4_3.5x3.5mm_P1.75mm, symbol LED:SK6812MINI
- removed D96: EnterRGB, LED_SMD:LED_SK6812MINI_PLCC4_3.5x3.5mm_P1.75mm, symbol LED:SK6812MINI
- removed D97: DeleteRGB, LED_SMD:LED_SK6812MINI_PLCC4_3.5x3.5mm_P1.75mm, symbol LED:SK6812MINI
- removed D98: PgDnRGB, LED_SMD:LED_SK6812MINI_PLCC4_3.5x3.5mm_P1.75mm, symbol LED:SK6812MINI
- removed SW1: ESC, marbastlib-mx:SW_MX_1u, symbol Switch:SW_Push
- removed SW10: F8, marbastlib-mx:SW_MX_1u, symbol Switch:SW_Push
- removed SW11: F9, marbastlib-mx:SW_MX_1u, symbol Switch:SW_Push
- removed SW12: F10, marbastlib-mx:SW_MX_1u, symbol Switch:SW_Push
- removed SW13: F11, marbastlib-mx:SW_MX_1u, symbol Switch:SW_Push
- removed SW14: F12, marbastlib-mx:SW_MX_1u, symbol Switch:SW_Push
- removed SW15: U1, marbastlib-mx:SW_MX_1u, symbol Switch:SW_Push
- removed SW16: PrtSc, marbastlib-mx:SW_MX_1u, symbol Switch:SW_Push
- removed SW17: PauseBr, marbastlib-mx:SW_MX_1u, symbol Switch:SW_Push
- removed SW18: `, marbastlib-mx:SW_MX_1u, symbol Switch:SW_Push
- removed SW19: #1, marbastlib-mx:SW_MX_1u, symbol Switch:SW_Push
- removed SW2: F1, marbastlib-mx:SW_MX_1u, symbol Switch:SW_Push
- removed SW20: #2, marbastlib-mx:SW_MX_1u, symbol Switch:SW_Push
- removed SW21: #3, marbastlib-mx:SW_MX_1u, symbol Switch:SW_Push
- removed SW22: #4, marbastlib-mx:SW_MX_1u, symbol Switch:SW_Push
- removed SW23: #5, marbastlib-mx:SW_MX_1u, symbol Switch:SW_Push
- removed SW24: #6, marbastlib-mx:SW_MX_1u, symbol Switch:SW_Push
- removed SW25: #7, marbastlib-mx:SW_MX_1u, symbol Switch:SW_Push
- removed SW26: #8, marbastlib-mx:SW_MX_1u, symbol Switch:SW_Push
- removed SW27: #9, marbastlib-mx:SW_MX_1u, symbol Switch:SW_Push
- removed SW28: #0, marbastlib-mx:SW_MX_1u, symbol Switch:SW_Push
- removed SW29: -, marbastlib-mx:SW_MX_1u, symbol Switch:SW_Push
- removed SW3: F2, marbastlib-mx:SW_MX_1u, symbol Switch:SW_Push
- removed SW30: =, marbastlib-mx:SW_MX_1u, symbol Switch:SW_Push
- removed SW31: BackSpace, marbastlib-mx:SW_MX_1u, symbol Switch:SW_Push
- removed SW32: Insert, marbastlib-mx:SW_MX_1u, symbol Switch:SW_Push
- removed SW33: PgUp, marbastlib-mx:SW_MX_1u, symbol Switch:SW_Push
- removed SW34: Tab, marbastlib-mx:SW_MX_1.5u, symbol Switch:SW_Push
- removed SW35: Q, marbastlib-mx:SW_MX_1u, symbol Switch:SW_Push
- removed SW36: W, marbastlib-mx:SW_MX_1u, symbol Switch:SW_Push
- removed SW37: E, marbastlib-mx:SW_MX_1u, symbol Switch:SW_Push
- removed SW38: R, marbastlib-mx:SW_MX_1u, symbol Switch:SW_Push
- removed SW39: T, marbastlib-mx:SW_MX_1u, symbol Switch:SW_Push
- removed SW4: F3, marbastlib-mx:SW_MX_1u, symbol Switch:SW_Push
- removed SW40: Y, marbastlib-mx:SW_MX_1u, symbol Switch:SW_Push
- removed SW41: U, marbastlib-mx:SW_MX_1u, symbol Switch:SW_Push
- removed SW42: I, marbastlib-mx:SW_MX_1u, symbol Switch:SW_Push
- removed SW43: O, marbastlib-mx:SW_MX_1u, symbol Switch:SW_Push
- removed SW44: P, marbastlib-mx:SW_MX_1u, symbol Switch:SW_Push
- removed SW45: [, marbastlib-mx:SW_MX_1u, symbol Switch:SW_Push
- removed SW46: ], marbastlib-mx:SW_MX_1u, symbol Switch:SW_Push
- removed SW47: Enter, marbastlib-mx:SW_MX_1u, symbol Switch:SW_Push
- removed SW48: Delete, marbastlib-mx:SW_MX_1u, symbol Switch:SW_Push
- removed SW49: PgDn, marbastlib-mx:SW_MX_1u, symbol Switch:SW_Push
- removed SW5: F4, marbastlib-mx:SW_MX_1u, symbol Switch:SW_Push
- removed SW50: CapsLock, marbastlib-mx:SW_MX_1.75u, symbol Switch:SW_Push
- removed SW51: A, marbastlib-mx:SW_MX_1u, symbol Switch:SW_Push
- removed SW52: S, marbastlib-mx:SW_MX_1u, symbol Switch:SW_Push
- removed SW53: D, marbastlib-mx:SW_MX_1u, symbol Switch:SW_Push
- removed SW54: F, marbastlib-mx:SW_MX_1u, symbol Switch:SW_Push
- removed SW55: G, marbastlib-mx:SW_MX_1u, symbol Switch:SW_Push
- removed SW56: H, marbastlib-mx:SW_MX_1u, symbol Switch:SW_Push
- removed SW57: J, marbastlib-mx:SW_MX_1u, symbol Switch:SW_Push
- removed SW58: K, marbastlib-mx:SW_MX_1u, symbol Switch:SW_Push
- removed SW59: L, marbastlib-mx:SW_MX_1u, symbol Switch:SW_Push
- removed SW6: F5, marbastlib-mx:SW_MX_1u, symbol Switch:SW_Push
- removed SW60: ;, marbastlib-mx:SW_MX_1u, symbol Switch:SW_Push
- removed SW61: '@, marbastlib-mx:SW_MX_1u, symbol Switch:SW_Push
- removed SW62: #~, marbastlib-mx:SW_MX_1u, symbol Switch:SW_Push
- removed SW63: Home, marbastlib-mx:SW_MX_1u, symbol Switch:SW_Push
- removed SW64: End, marbastlib-mx:SW_MX_1u, symbol Switch:SW_Push
- removed SW65: LShift, marbastlib-mx:SW_MX_1.25u, symbol Switch:SW_Push
- removed SW66: \|, marbastlib-mx:SW_MX_1u, symbol Switch:SW_Push
- removed SW67: Z, marbastlib-mx:SW_MX_1u, symbol Switch:SW_Push
- removed SW68: X, marbastlib-mx:SW_MX_1u, symbol Switch:SW_Push
- removed SW69: C, marbastlib-mx:SW_MX_1u, symbol Switch:SW_Push
- removed SW7: F6, marbastlib-mx:SW_MX_1u, symbol Switch:SW_Push
- removed SW70: V, marbastlib-mx:SW_MX_1u, symbol Switch:SW_Push
- removed SW71: B, marbastlib-mx:SW_MX_1u, symbol Switch:SW_Push
- removed SW72: N, marbastlib-mx:SW_MX_1u, symbol Switch:SW_Push
- removed SW73: M, marbastlib-mx:SW_MX_1u, symbol Switch:SW_Push
- removed SW74: ,<, marbastlib-mx:SW_MX_1u, symbol Switch:SW_Push
- removed SW75: .>, marbastlib-mx:SW_MX_1u, symbol Switch:SW_Push
- removed SW76: /?, marbastlib-mx:SW_MX_1u, symbol Switch:SW_Push
- removed SW77: RShift, marbastlib-mx:SW_MX_1.75u, symbol Switch:SW_Push
- removed SW78: UpArrow, marbastlib-mx:SW_MX_1u, symbol Switch:SW_Push
- removed SW79: U2, marbastlib-mx:SW_MX_1u, symbol Switch:SW_Push
- removed SW8: XEV, marbastlib-mx:SW_MX_1u, symbol Switch:SW_Push
- removed SW80: U3, marbastlib-mx:SW_MX_1u, symbol Switch:SW_Push
- removed SW81: LCtrl, marbastlib-mx:SW_MX_1.25u, symbol Switch:SW_Push
- removed SW82: Win, marbastlib-mx:SW_MX_1.25u, symbol Switch:SW_Push
- removed SW83: Alt, marbastlib-mx:SW_MX_1.25u, symbol Switch:SW_Push
- removed SW84: Space, marbastlib-mx:SW_MX_1u, symbol Switch:SW_Push
- removed SW85: AltGr, marbastlib-mx:SW_MX_1u, symbol Switch:SW_Push
- removed SW86: Fn, marbastlib-mx:SW_MX_1u, symbol Switch:SW_Push
- removed SW87: RCtrl, marbastlib-mx:SW_MX_1u, symbol Switch:SW_Push
- removed SW88: LeftArrow, marbastlib-mx:SW_MX_1u, symbol Switch:SW_Push
- removed SW89: DownArrow, marbastlib-mx:SW_MX_1u, symbol Switch:SW_Push
- removed SW9: F7, marbastlib-mx:SW_MX_1u, symbol Switch:SW_Push
- removed SW90: RightArrow, marbastlib-mx:SW_MX_1u, symbol Switch:SW_Push
- removed SW91: U4, marbastlib-mx:SW_MX_1u, symbol Switch:SW_Push
- added D18, D19, D20, D21, D22, D23, D24, D25, D26, D27, D28, D29, D30, D31, D32, D33, D34, D51, D52, D53, D54, D55, D56, D57, D58, D59, D60, D61, D62, D63, D64, D65, D66, D83, D84, D85, D86, D87, D88, D89, D90, D91: D_Small, Diode_SMD:D_SOD-123, symbol Device:D_Small
- added LED1, LED10, LED11, LED12, LED13, LED14, LED15, LED16, LED17, LED18, LED19, LED2, LED20, LED21, LED22, LED23, LED24, LED25, LED26, LED27, LED28, LED29, LED3, LED30, LED31, LED32, LED33, LED34, LED35, LED36, LED37, LED38, LED39, LED4, LED40, LED41, LED42, LED43, LED44, LED45, LED46, LED47, LED48, LED49, LED5, LED50, LED51, LED52, LED53, LED54, LED55, LED56, LED57, LED58, LED59, LED6, LED60, LED61, LED62, LED63, LED64, LED65, LED66, LED67, LED68, LED69, LED7, LED70, LED71, LED72, LED73, LED74, LED75, LED76, LED77, LED78, LED79, LED8, LED80, LED81, LED82, LED83, LED84, LED85, LED86, LED87, LED88, LED89, LED9, LED90, LED91: MX_SK6812MINI-E, marbastlib-mx:LED_MX_6028R, symbol marbastlib-mx:MX_SK6812MINI-E
- added SW1: Esc, marbastlib-mx:SW_MX_1u, symbol marbastlib-mx:MX_SW_solder
- added SW10: #F8, marbastlib-mx:SW_MX_1u, symbol marbastlib-mx:MX_SW_solder
- added SW11: #F9, marbastlib-mx:SW_MX_1u, symbol marbastlib-mx:MX_SW_solder
- added SW12: #F10, marbastlib-mx:SW_MX_1u, symbol marbastlib-mx:MX_SW_solder
- added SW13: #F11, marbastlib-mx:SW_MX_1u, symbol marbastlib-mx:MX_SW_solder
- added SW14: #F12, marbastlib-mx:SW_MX_1u, symbol marbastlib-mx:MX_SW_solder
- added SW15: U5, marbastlib-mx:SW_MX_1u, symbol marbastlib-mx:MX_SW_solder
- added SW16: PrtSc, marbastlib-mx:SW_MX_1u, symbol marbastlib-mx:MX_SW_solder
- added SW17: PauseBreak, marbastlib-mx:SW_MX_1u, symbol marbastlib-mx:MX_SW_solder
- added SW18: `, marbastlib-mx:SW_MX_1u, symbol marbastlib-mx:MX_SW_solder
- added SW19: #1, marbastlib-mx:SW_MX_1u, symbol marbastlib-mx:MX_SW_solder
- added SW2: #F1, marbastlib-mx:SW_MX_1u, symbol marbastlib-mx:MX_SW_solder
- added SW20: #2, marbastlib-mx:SW_MX_1u, symbol marbastlib-mx:MX_SW_solder
- added SW21: #3, marbastlib-mx:SW_MX_1u, symbol marbastlib-mx:MX_SW_solder
- added SW22: #4, marbastlib-mx:SW_MX_1u, symbol marbastlib-mx:MX_SW_solder
- added SW23: #5, marbastlib-mx:SW_MX_1u, symbol marbastlib-mx:MX_SW_solder
- added SW24: #6, marbastlib-mx:SW_MX_1u, symbol marbastlib-mx:MX_SW_solder
- added SW25: #7, marbastlib-mx:SW_MX_1u, symbol marbastlib-mx:MX_SW_solder
- added SW26: #8, marbastlib-mx:SW_MX_1u, symbol marbastlib-mx:MX_SW_solder
- added SW27: #9, marbastlib-mx:SW_MX_1u, symbol marbastlib-mx:MX_SW_solder
- added SW28: #0, marbastlib-mx:SW_MX_1u, symbol marbastlib-mx:MX_SW_solder
- added SW29: -, marbastlib-mx:SW_MX_1u, symbol marbastlib-mx:MX_SW_solder
- added SW3: #F2, marbastlib-mx:SW_MX_1u, symbol marbastlib-mx:MX_SW_solder
- added SW30: =, marbastlib-mx:SW_MX_1u, symbol marbastlib-mx:MX_SW_solder
- added SW31: BackSpace, marbastlib-mx:SW_MX_1u, symbol marbastlib-mx:MX_SW_solder
- added SW32: Insert, marbastlib-mx:SW_MX_1u, symbol marbastlib-mx:MX_SW_solder
- added SW33: PgUp, marbastlib-mx:SW_MX_1u, symbol marbastlib-mx:MX_SW_solder
- added SW34: Tab, marbastlib-mx:SW_MX_1.5u, symbol marbastlib-mx:MX_SW_solder
- added SW35: Q, marbastlib-mx:SW_MX_1u, symbol marbastlib-mx:MX_SW_solder
- added SW36: W, marbastlib-mx:SW_MX_1u, symbol marbastlib-mx:MX_SW_solder
- added SW37: #E, marbastlib-mx:SW_MX_1u, symbol marbastlib-mx:MX_SW_solder
- added SW38: #R, marbastlib-mx:SW_MX_1u, symbol marbastlib-mx:MX_SW_solder
- added SW39: T, marbastlib-mx:SW_MX_1u, symbol marbastlib-mx:MX_SW_solder
- added SW4: #F3, marbastlib-mx:SW_MX_1u, symbol marbastlib-mx:MX_SW_solder
- added SW40: Y, marbastlib-mx:SW_MX_1u, symbol marbastlib-mx:MX_SW_solder
- added SW41: U, marbastlib-mx:SW_MX_1u, symbol marbastlib-mx:MX_SW_solder
- added SW42: I, marbastlib-mx:SW_MX_1u, symbol marbastlib-mx:MX_SW_solder
- added SW43: O, marbastlib-mx:SW_MX_1u, symbol marbastlib-mx:MX_SW_solder
- added SW44: P, marbastlib-mx:SW_MX_1u, symbol marbastlib-mx:MX_SW_solder
- added SW45: [, marbastlib-mx:SW_MX_1u, symbol marbastlib-mx:MX_SW_solder
- added SW46: ], marbastlib-mx:SW_MX_1u, symbol marbastlib-mx:MX_SW_solder
- added SW47: Enter, marbastlib-mx:SW_MX_1u, symbol marbastlib-mx:MX_SW_solder
- added SW48: Delete, marbastlib-mx:SW_MX_1u, symbol marbastlib-mx:MX_SW_solder
- added SW49: PgDn, marbastlib-mx:SW_MX_1u, symbol marbastlib-mx:MX_SW_solder
- added SW5: #F4, marbastlib-mx:SW_MX_1u, symbol marbastlib-mx:MX_SW_solder
- added SW50: CapsLock, marbastlib-mx:SW_MX_1.75u, symbol marbastlib-mx:MX_SW_solder
- added SW51: #A, marbastlib-mx:SW_MX_1u, symbol marbastlib-mx:MX_SW_solder
- added SW52: S, marbastlib-mx:SW_MX_1u, symbol marbastlib-mx:MX_SW_solder
- added SW53: #D, marbastlib-mx:SW_MX_1u, symbol marbastlib-mx:MX_SW_solder
- added SW54: #F, marbastlib-mx:SW_MX_1u, symbol marbastlib-mx:MX_SW_solder
- added SW55: G, marbastlib-mx:SW_MX_1u, symbol marbastlib-mx:MX_SW_solder
- added SW56: H, marbastlib-mx:SW_MX_1u, symbol marbastlib-mx:MX_SW_solder
- added SW57: J, marbastlib-mx:SW_MX_1u, symbol marbastlib-mx:MX_SW_solder
- added SW58: K, marbastlib-mx:SW_MX_1u, symbol marbastlib-mx:MX_SW_solder
- added SW59: L, marbastlib-mx:SW_MX_1u, symbol marbastlib-mx:MX_SW_solder
- added SW6: #F5, marbastlib-mx:SW_MX_1u, symbol marbastlib-mx:MX_SW_solder
- added SW60: ;:, marbastlib-mx:SW_MX_1u, symbol marbastlib-mx:MX_SW_solder
- added SW61: '@, marbastlib-mx:SW_MX_1u, symbol marbastlib-mx:MX_SW_solder
- added SW62: ~#, marbastlib-mx:SW_MX_1u, symbol marbastlib-mx:MX_SW_solder
- added SW63: Home, marbastlib-mx:SW_MX_1u, symbol marbastlib-mx:MX_SW_solder
- added SW64: End, marbastlib-mx:SW_MX_1u, symbol marbastlib-mx:MX_SW_solder
- added SW65: LShift, marbastlib-mx:SW_MX_1.25u, symbol marbastlib-mx:MX_SW_solder
- added SW66: \|, marbastlib-mx:SW_MX_1u, symbol marbastlib-mx:MX_SW_solder
- added SW67: Z, marbastlib-mx:SW_MX_1u, symbol marbastlib-mx:MX_SW_solder
- added SW68: X, marbastlib-mx:SW_MX_1u, symbol marbastlib-mx:MX_SW_solder
- added SW69: #C, marbastlib-mx:SW_MX_1u, symbol marbastlib-mx:MX_SW_solder
- added SW7: #F6, marbastlib-mx:SW_MX_1u, symbol marbastlib-mx:MX_SW_solder
- added SW70: V, marbastlib-mx:SW_MX_1u, symbol marbastlib-mx:MX_SW_solder
- added SW71: B, marbastlib-mx:SW_MX_1u, symbol marbastlib-mx:MX_SW_solder
- added SW72: N, marbastlib-mx:SW_MX_1u, symbol marbastlib-mx:MX_SW_solder
- added SW73: M, marbastlib-mx:SW_MX_1u, symbol marbastlib-mx:MX_SW_solder
- added SW74: ,<, marbastlib-mx:SW_MX_1u, symbol marbastlib-mx:MX_SW_solder
- added SW75: .>, marbastlib-mx:SW_MX_1u, symbol marbastlib-mx:MX_SW_solder
- added SW76: /?, marbastlib-mx:SW_MX_1u, symbol marbastlib-mx:MX_SW_solder
- added SW77: RShift, marbastlib-mx:SW_MX_1.75u, symbol marbastlib-mx:MX_SW_solder
- added SW78: UpArrow, marbastlib-mx:SW_MX_1u, symbol marbastlib-mx:MX_SW_solder
- added SW79: U2, marbastlib-mx:SW_MX_1u, symbol marbastlib-mx:MX_SW_solder
- added SW8: XEV, marbastlib-mx:SW_MX_1u, symbol marbastlib-mx:MX_SW_solder
- added SW80: U3, marbastlib-mx:SW_MX_1u, symbol marbastlib-mx:MX_SW_solder
- added SW81: LCtrl, marbastlib-mx:SW_MX_1.25u, symbol marbastlib-mx:MX_SW_solder
- added SW82: Win, marbastlib-mx:SW_MX_1.25u, symbol marbastlib-mx:MX_SW_solder
- added SW83: Alt, marbastlib-mx:SW_MX_1.25u, symbol marbastlib-mx:MX_SW_solder
- added SW84: Space, marbastlib-mx:SW_MX_1u, symbol marbastlib-mx:MX_SW_solder
- added SW85: AltGr, marbastlib-mx:SW_MX_1u, symbol marbastlib-mx:MX_SW_solder
- added SW86: Fn, marbastlib-mx:SW_MX_1u, symbol marbastlib-mx:MX_SW_solder
- added SW87: RCtrl, marbastlib-mx:SW_MX_1u, symbol marbastlib-mx:MX_SW_solder
- added SW88: LeftArrow, marbastlib-mx:SW_MX_1u, symbol marbastlib-mx:MX_SW_solder
- added SW89: DownArrow, marbastlib-mx:SW_MX_1u, symbol marbastlib-mx:MX_SW_solder
- added SW9: #F7, marbastlib-mx:SW_MX_1u, symbol marbastlib-mx:MX_SW_solder
- added SW90: RightArrow, marbastlib-mx:SW_MX_1u, symbol marbastlib-mx:MX_SW_solder
- added SW91: U4, marbastlib-mx:SW_MX_1u, symbol marbastlib-mx:MX_SW_solder
Connections:
- net GND: now also LED1.4 (VSS), LED10.4 (VSS), LED11.4 (VSS), LED12.4 (VSS), LED13.4 (VSS), LED14.4 (VSS), LED15.4 (VSS), LED16.4 (VSS), LED17.4 (VSS), LED18.4 (VSS), LED19.4 (VSS), LED2.4 (VSS), LED20.4 (VSS), LED21.4 (VSS), LED22.4 (VSS), LED23.4 (VSS), LED24.4 (VSS), LED25.4 (VSS), LED26.4 (VSS), LED27.4 (VSS), LED28.4 (VSS), LED29.4 (VSS), LED3.4 (VSS), LED30.4 (VSS), LED31.4 (VSS), LED32.4 (VSS), LED33.4 (VSS), LED34.4 (VSS), LED35.4 (VSS), LED36.4 (VSS), LED37.4 (VSS), LED38.4 (VSS), LED39.4 (VSS), LED4.4 (VSS), LED40.4 (VSS), LED41.4 (VSS), LED42.4 (VSS), LED43.4 (VSS), LED44.4 (VSS), LED45.4 (VSS), LED46.4 (VSS), LED47.4 (VSS), LED48.4 (VSS), LED49.4 (VSS), LED5.4 (VSS), LED50.4 (VSS), LED51.4 (VSS), LED52.4 (VSS), LED53.4 (VSS), LED54.4 (VSS), LED55.4 (VSS), LED56.4 (VSS), LED57.4 (VSS), LED58.4 (VSS), LED59.4 (VSS), LED6.4 (VSS), LED60.4 (VSS), LED61.4 (VSS), LED62.4 (VSS), LED63.4 (VSS), LED64.4 (VSS), LED65.4 (VSS), LED66.4 (VSS), LED67.4 (VSS), LED68.4 (VSS), LED69.4 (VSS), LED7.4 (VSS), LED70.4 (VSS), LED71.4 (VSS), LED72.4 (VSS), LED73.4 (VSS), LED74.4 (VSS), LED75.4 (VSS), LED76.4 (VSS), LED77.4 (VSS), LED78.4 (VSS), LED79.4 (VSS), LED8.4 (VSS), LED80.4 (VSS), LED81.4 (VSS), LED82.4 (VSS), LED83.4 (VSS), LED84.4 (VSS), LED85.4 (VSS), LED86.4 (VSS), LED87.4 (VSS), LED88.4 (VSS), LED89.4 (VSS), LED9.4 (VSS), LED90.4 (VSS), LED91.4 (VSS)
- net VCC: now also LED1.1 (VDD), LED10.1 (VDD), LED11.1 (VDD), LED12.1 (VDD), LED13.1 (VDD), LED14.1 (VDD), LED15.1 (VDD), LED16.1 (VDD), LED17.1 (VDD), LED18.1 (VDD), LED19.1 (VDD), LED2.1 (VDD), LED20.1 (VDD), LED21.1 (VDD), LED22.1 (VDD), LED23.1 (VDD), LED24.1 (VDD), LED25.1 (VDD), LED26.1 (VDD), LED27.1 (VDD), LED28.1 (VDD), LED29.1 (VDD), LED3.1 (VDD), LED30.1 (VDD), LED31.1 (VDD), LED32.1 (VDD), LED33.1 (VDD), LED34.1 (VDD), LED35.1 (VDD), LED36.1 (VDD), LED37.1 (VDD), LED38.1 (VDD), LED39.1 (VDD), LED4.1 (VDD), LED40.1 (VDD), LED41.1 (VDD), LED42.1 (VDD), LED43.1 (VDD), LED44.1 (VDD), LED45.1 (VDD), LED46.1 (VDD), LED47.1 (VDD), LED48.1 (VDD), LED49.1 (VDD), LED5.1 (VDD), LED50.1 (VDD), LED51.1 (VDD), LED52.1 (VDD), LED53.1 (VDD), LED54.1 (VDD), LED55.1 (VDD), LED56.1 (VDD), LED57.1 (VDD), LED58.1 (VDD), LED59.1 (VDD), LED6.1 (VDD), LED60.1 (VDD), LED61.1 (VDD), LED62.1 (VDD), LED63.1 (VDD), LED64.1 (VDD), LED65.1 (VDD), LED66.1 (VDD), LED67.1 (VDD), LED68.1 (VDD), LED69.1 (VDD), LED7.1 (VDD), LED70.1 (VDD), LED71.1 (VDD), LED72.1 (VDD), LED73.1 (VDD), LED74.1 (VDD), LED75.1 (VDD), LED76.1 (VDD), LED77.1 (VDD), LED78.1 (VDD), LED79.1 (VDD), LED8.1 (VDD), LED80.1 (VDD), LED81.1 (VDD), LED82.1 (VDD), LED83.1 (VDD), LED84.1 (VDD), LED85.1 (VDD), LED86.1 (VDD), LED87.1 (VDD), LED88.1 (VDD), LED89.1 (VDD), LED9.1 (VDD), LED90.1 (VDD), LED91.1 (VDD)
- net col0: now also SW1.1, SW18.1, SW34.1, SW50.1, SW65.1, SW81.1
- net col1: now also SW19.1, SW2.1, SW35.1, SW51.1, SW66.1, SW82.1
- net col10: now also SW11.1, SW28.1, SW44.1, SW60.1, SW75.1, SW85.1
- net col11: now also SW12.1, SW29.1, SW45.1, SW61.1, SW76.1, SW86.1
- net col12: now also SW13.1, SW30.1, SW46.1, SW62.1, SW77.1, SW87.1
- net col13: now also SW14.1, SW31.1, SW47.1, SW78.1, SW88.1
- net col14: now also SW15.1, SW89.1
- net col15: now also SW16.1, SW32.1, SW48.1, SW63.1, SW79.1, SW90.1
- net col16: now also SW17.1, SW33.1, SW49.1, SW64.1, SW80.1, SW91.1
- net col2: now also SW20.1, SW3.1, SW36.1, SW52.1, SW67.1, SW83.1
- net col3: now also SW21.1, SW37.1, SW4.1, SW53.1, SW68.1
- net col4: now also SW22.1, SW38.1, SW5.1, SW54.1, SW69.1
- net col5: now also SW23.1, SW39.1, SW55.1, SW6.1, SW70.1
- net col6: now also SW24.1, SW40.1, SW56.1, SW7.1, SW71.1, SW84.1
- net col7: now also SW25.1, SW41.1, SW57.1, SW72.1, SW8.1
- net col8: now also SW26.1, SW42.1, SW58.1, SW73.1, SW9.1
- net col9: now also SW10.1, SW27.1, SW43.1, SW59.1, SW74.1
- net led: now also LED1.3 (DIN)
- net row1: now also D18.1 (K), D19.1 (K), D20.1 (K), D21.1 (K), D22.1 (K), D23.1 (K), D24.1 (K), D25.1 (K), D26.1 (K), D27.1 (K), D28.1 (K), D29.1 (K), D30.1 (K), D31.1 (K), D32.1 (K), D33.1 (K); no longer D35.1 (K), D36.1 (K), D37.1 (K), D38.1 (K), D39.1 (K), D40.1 (K), D41.1 (K), D42.1 (K), D43.1 (K), D44.1 (K), D45.1 (K), D46.1 (K), D47.1 (K), D48.1 (K), D49.1 (K), D50.1 (K)
- net row2: now also D35.1 (K), D36.1 (K), D37.1 (K), D38.1 (K), D39.1 (K), D40.1 (K), D41.1 (K), D42.1 (K), D43.1 (K), D44.1 (K), D45.1 (K), D46.1 (K), D47.1 (K), D48.1 (K), D49.1 (K), D34.1 (K); no longer D67.1 (K), D68.1 (K), D69.1 (K), D70.1 (K), D71.1 (K), D72.1 (K), D73.1 (K), D74.1 (K), D75.1 (K), D76.1 (K), D77.1 (K), D78.1 (K), D79.1 (K), D80.1 (K), D81.1 (K), D82.1 (K)
- net row3: now also D50.1 (K), D51.1 (K), D52.1 (K), D53.1 (K), D54.1 (K), D55.1 (K), D56.1 (K), D57.1 (K), D58.1 (K), D59.1 (K), D60.1 (K), D61.1 (K), D62.1 (K), D63.1 (K), D64.1 (K)
- net row4: now also D67.1 (K), D68.1 (K), D69.1 (K), D70.1 (K), D71.1 (K), D72.1 (K), D73.1 (K), D74.1 (K), D75.1 (K), D76.1 (K), D77.1 (K), D78.1 (K), D79.1 (K), D80.1 (K), D65.1 (K), D66.1 (K)
- net row5: now also D81.1 (K), D82.1 (K), D83.1 (K), D84.1 (K), D85.1 (K), D86.1 (K), D87.1 (K), D88.1 (K), D89.1 (K), D90.1 (K), D91.1 (K)
- net at D49.2 (A): now also SW49.2
- net at D80.2 (A): now also SW80.2
- net at D73.2 (A): now also SW73.2
- net at D42.2 (A): now also SW42.2
- net at D74.2 (A): now also SW74.2
- net at D77.2 (A): now also SW77.2
- net at D16.2 (A): now also SW16.2
- net at D39.2 (A): now also SW39.2
- net at D10.2 (A): now also SW10.2
- net at D7.2 (A): now also SW7.2
- net at D46.2 (A): now also SW46.2
- net at D5.2 (A): now also SW5.2
- net at D68.2 (A): now also SW68.2
- net at D47.2 (A): now also SW47.2
- net at D14.2 (A): now also SW14.2
- net at D44.2 (A): now also SW44.2
- net at D2.2 (A): now also SW2.2
- net at D41.2 (A): now also SW41.2
- net at D1.2 (A): now also SW1.2
- net at D40.2 (A): now also SW40.2
- net at D72.2 (A): now also SW72.2
- net at D71.2 (A): now also SW71.2
- net at D38.2 (A): now also SW38.2
- net at D79.2 (A): now also SW79.2
- net at D13.2 (A): now also SW13.2
- net at D78.2 (A): now also SW78.2
- net at D82.2 (A): now also SW82.2
- net at D37.2 (A): now also SW37.2
- net at D75.2 (A): now also SW75.2
- net at D8.2 (A): now also SW8.2
- net at D12.2 (A): now also SW12.2
- net at D35.2 (A): now also SW35.2
- net at D69.2 (A): now also SW69.2
- net at D3.2 (A): now also SW3.2
- net at D11.2 (A): now also SW11.2
- net at D6.2 (A): now also SW6.2
- net at D76.2 (A): now also SW76.2
- net at D9.2 (A): now also SW9.2
- net at D81.2 (A): now also SW81.2
- net at D70.2 (A): now also SW70.2
- net at D43.2 (A): now also SW43.2
- net at D45.2 (A): now also SW45.2
- net at D36.2 (A): now also SW36.2
- net at D48.2 (A): now also SW48.2
- net at D67.2 (A): now also SW67.2
- net at D15.2 (A): now also SW15.2
- net at D4.2 (A): now also SW4.2
- net at D17.2 (A): now also SW17.2
- net at D50.2 (A): now also SW50.2
- new net: D66.2 (A), SW66.2
- new net: LED12.2 (DOUT), LED13.3 (DIN)
- new net: LED11.2 (DOUT), LED12.3 (DIN)
- new net: D34.2 (A), SW34.2
- new net: D19.2 (A), SW19.2
- new net: D61.2 (A), SW61.2
- new net: LED19.2 (DOUT), LED20.3 (DIN)
- new net: LED18.2 (DOUT), LED19.3 (DIN)
- new net: D21.2 (A), SW21.2
- new net: LED88.2 (DOUT), LED89.3 (DIN)
- new net: LED87.2 (DOUT), LED88.3 (DIN)
- new net: LED10.2 (DOUT), LED11.3 (DIN)
- new net: LED83.2 (DOUT), LED84.3 (DIN)
- new net: LED82.2 (DOUT), LED83.3 (DIN)
- new net: LED72.2 (DOUT), LED73.3 (DIN)
- new net: LED71.2 (DOUT), LED72.3 (DIN)
- new net: LED46.2 (DOUT), LED47.3 (DIN)
- new net: LED45.2 (DOUT), LED46.3 (DIN)
- new net: D32.2 (A), SW32.2
- new net: D56.2 (A), SW56.2
- new net: D60.2 (A), SW60.2
- new net: LED29.2 (DOUT), LED30.3 (DIN)
- new net: LED28.2 (DOUT), LED29.3 (DIN)
- new net: LED52.2 (DOUT), LED53.3 (DIN)
- new net: LED51.2 (DOUT), LED52.3 (DIN)
- new net: LED79.2 (DOUT), LED80.3 (DIN)
- new net: LED78.2 (DOUT), LED79.3 (DIN)
- new net: D26.2 (A), SW26.2
- new net: D18.2 (A), SW18.2
- new net: LED84.2 (DOUT), LED85.3 (DIN)
- new net: LED62.2 (DOUT), LED63.3 (DIN)
- new net: LED61.2 (DOUT), LED62.3 (DIN)
- new net: LED17.2 (DOUT), LED18.3 (DIN)
- new net: LED16.2 (DOUT), LED17.3 (DIN)
- new net: LED30.2 (DOUT), LED31.3 (DIN)
- new net: D29.2 (A), SW29.2
- new net: D91.2 (A), SW91.2
- new net: LED24.2 (DOUT), LED25.3 (DIN)
- new net: LED23.2 (DOUT), LED24.3 (DIN)
- new net: LED43.2 (DOUT), LED44.3 (DIN)
- new net: LED42.2 (DOUT), LED43.3 (DIN)
- new net: LED68.2 (DOUT), LED69.3 (DIN)
- new net: LED67.2 (DOUT), LED68.3 (DIN)
- new net: LED53.2 (DOUT), LED54.3 (DIN)
- new net: LED41.2 (DOUT), LED42.3 (DIN)
- new net: D65.2 (A), SW65.2
- new net: LED90.2 (DOUT), LED91.3 (DIN)
- new net: LED20.2 (DOUT), LED21.3 (DIN)
- new net: LED10.3 (DIN), LED9.2 (DOUT)
- new net: LED8.2 (DOUT), LED9.3 (DIN)
- new net: LED74.2 (DOUT), LED75.3 (DIN)
- new net: LED73.2 (DOUT), LED74.3 (DIN)
- new net: LED89.2 (DOUT), LED90.3 (DIN)
- new net: LED64.2 (DOUT), LED65.3 (DIN)
- new net: LED63.2 (DOUT), LED64.3 (DIN)
- new net: LED34.2 (DOUT), LED35.3 (DIN)
- new net: LED33.2 (DOUT), LED34.3 (DIN)
- new net: D25.2 (A), SW25.2
- new net: LED5.2 (DOUT), LED6.3 (DIN)
- new net: LED4.2 (DOUT), LED5.3 (DIN)
- new net: D87.2 (A), SW87.2
- new net: D57.2 (A), SW57.2
- new net: D20.2 (A), SW20.2
- new net: D85.2 (A), SW85.2
- new net: D64.2 (A), SW64.2
- new net: D55.2 (A), SW55.2
- new net: LED54.2 (DOUT), LED55.3 (DIN)
- new net: D83.2 (A), SW83.2
- new net: LED77.2 (DOUT), LED78.3 (DIN)
- new net: LED48.2 (DOUT), LED49.3 (DIN)
- new net: LED47.2 (DOUT), LED48.3 (DIN)
- new net: D52.2 (A), SW52.2
- new net: LED15.2 (DOUT), LED16.3 (DIN)
- new net: LED14.2 (DOUT), LED15.3 (DIN)
- new net: LED55.2 (DOUT), LED56.3 (DIN)
- new net: LED86.2 (DOUT), LED87.3 (DIN)
- new net: LED6.2 (DOUT), LED7.3 (DIN)
- new net: LED13.2 (DOUT), LED14.3 (DIN)
- new net: D62.2 (A), SW62.2
- new net: LED70.2 (DOUT), LED71.3 (DIN)
- new net: LED69.2 (DOUT), LED70.3 (DIN)
- new net: LED21.2 (DOUT), LED22.3 (DIN)
- new net: LED50.2 (DOUT), LED51.3 (DIN)
- new net: D89.2 (A), SW89.2
- new net: D28.2 (A), SW28.2
- new net: LED49.2 (DOUT), LED50.3 (DIN)
- new net: LED56.2 (DOUT), LED57.3 (DIN)
- new net: LED59.2 (DOUT), LED60.3 (DIN)
- new net: LED58.2 (DOUT), LED59.3 (DIN)
- new net: D51.2 (A), SW51.2
- new net: LED66.2 (DOUT), LED67.3 (DIN)
- new net: LED65.2 (DOUT), LED66.3 (DIN)
- new net: LED32.2 (DOUT), LED33.3 (DIN)
- new net: LED31.2 (DOUT), LED32.3 (DIN)
- new net: LED76.2 (DOUT), LED77.3 (DIN)
- new net: LED75.2 (DOUT), LED76.3 (DIN)
- new net: D88.2 (A), SW88.2
- new net: D53.2 (A), SW53.2
- new net: D86.2 (A), SW86.2
- new net: D90.2 (A), SW90.2
- new net: D24.2 (A), SW24.2
- new net: D22.2 (A), SW22.2
- new net: D63.2 (A), SW63.2
- new net: LED7.2 (DOUT), LED8.3 (DIN)
- new net: LED44.2 (DOUT), LED45.3 (DIN)
- new net: LED27.2 (DOUT), LED28.3 (DIN)
- new net: LED26.2 (DOUT), LED27.3 (DIN)
- new net: LED25.2 (DOUT), LED26.3 (DIN)
- new net: LED40.2 (DOUT), LED41.3 (DIN)
- new net: LED38.2 (DOUT), LED39.3 (DIN)
- new net: LED37.2 (DOUT), LED38.3 (DIN)
- new net: LED80.2 (DOUT), LED81.3 (DIN)
- new net: D30.2 (A), SW30.2
- new net: LED57.2 (DOUT), LED58.3 (DIN)
- new net: D58.2 (A), SW58.2
- new net: D27.2 (A), SW27.2
- new net: D31.2 (A), SW31.2
- new net: LED22.2 (DOUT), LED23.3 (DIN)
- new net: LED3.2 (DOUT), LED4.3 (DIN)
- new net: LED2.2 (DOUT), LED3.3 (DIN)
- new net: D59.2 (A), SW59.2
- new net: D33.2 (A), SW33.2
- new net: D23.2 (A), SW23.2
- new net: LED1.2 (DOUT), LED2.3 (DIN)
- new net: LED35.2 (DOUT), LED36.3 (DIN)
- new net: LED39.2 (DOUT), LED40.3 (DIN)
- new net: D54.2 (A), SW54.2
- new net: LED85.2 (DOUT), LED86.3 (DIN)
- new net: D84.2 (A), SW84.2
- new net: LED36.2 (DOUT), LED37.3 (DIN)
- new net: LED60.2 (DOUT), LED61.3 (DIN)
- new net: LED81.2 (DOUT), LED82.3 (DIN)
