File: X95X/X95X.kicad_pcb (KiCad board)
At the start: 2 copper layers, 10.1 x 6.4 mm, 298 parts, among them J1 USB_C_Receptacle_USB2.0, J2 AVR-ISP-6, SW1 ESC, SW10 F8, SW11 F9, SW12 F10, SW13 F11, SW14 F12, SW15 U1, SW16 PrtSc, SW17 PauseBr, SW18 `, SW19 #1, SW2 F1, SW20 #2, SW21 #3, SW22 #4, SW23 #5, SW24 #6, SW25 #7, SW26 #8, SW27 #9, SW28 #0, SW29 -, SW3 F2, SW30 =, SW31 BackSpace, SW32 Insert, SW33 PgUp, SW34 Tab, SW35 Q, SW36 W, SW37 E, SW38 R, SW39 T, SW4 F3, SW40 Y, SW41 U, SW42 I, SW43 O, SW44 P, SW45 [, SW46 ], SW47 Enter, SW48 Delete, SW49 PgDn, SW5 F4, SW50 CapsLock, SW51 A, SW52 S, SW53 D, SW54 F, SW55 G, SW56 H, SW57 J, SW58 K, SW59 L, SW6 F5, SW60 ;, SW61 '@, SW62 #~, SW63 Home, SW64 End, SW65 LShift, SW66 \|, SW67 Z, SW68 X, SW69 C, SW7 F6, SW70 V, SW71 B, SW72 N, SW73 M, SW74 ,<, SW75 .>, SW76 /?, SW77 RShift, SW78 UpArrow, SW79 U2, SW8 XEV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

Commit message: more pcb
Parts:
- C1, C2, C3, C4, C5, C6, C7, C8, D1, D10, D100, D101, D102, D103, D104, D105, D106, D107, D108, D109, D11, D110, D111, D112, D113, D114, D115, D116, D117, D118, D119, D12, D120, D121, D122, D123, D124, D125, D126, D127, D128, D129, D13, D130, D131, D132, D133, D134, D135, D136, D137, D138, D139, D14, D140, D141, D142, D143, D144, D145, D146, D147, D148, D149, D15, D150, D151, D152, D153, D154, D155, D156, D157, D158, D159, D16, D160, D161, D162, D163, D164, D165, D166, D167, D168, D169, D17, D170, D171, D172, D173, D174, D175, D176, D177, D178, D179, D18, D180, D181, D182, D183, D19, D2, D20, D21, D22, D23, D24, D25, D26, D27, D28, D29, D3, D30, D31, D32, D33, D34, D35, D36, D37, D38, D39, D4, D40, D41, D42, D43, D44, D45, D46, D47, D48, D49, D5, D50, D51, D52, D53, D54, D55, D56, D57, D58, D59, D6, D60, D61, D62, D63, D64, D65, D66, D67, D68, D69, D7, D70, D71, D72, D73, D74, D75, D76, D77, D78, D79, D8, D80, D81, D82, D83, D84, D85, D86, D87, D88, D89, D9, D90, D91, D92, D93, D94, D95, D96, D97, D98, D99, F1, J1, J2, R1, R2, R3, R4, R5, R6, R7, SW92, U1, Y1: moved to B.Cu
- moved D50 325.4 mm to (34.0, -39.1), turned to 180 degrees
- moved D150 318.0 mm to (355.7, 143.3), turned to 180 degrees
- moved D104 313.9 mm to (39.7, -39.1), turned to 180 degrees
- moved D105 313.9 mm to (39.7, -35.8), turned to 180 degrees
- moved J1 311.6 mm to (352.5, 166.7), turned to 180 degrees
- moved U1 310.5 mm to (352.0, 157.2), turned to 180 degrees
- moved D115 303.9 mm to (348.7, 143.3), turned to 180 degrees
- moved D11 299.9 mm to (46.8, -34.1), turned to 180 degrees
- moved D39 299.9 mm to (46.8, -30.7), turned to 180 degrees
- moved D167 297.4 mm to (48.0, -27.4), turned to 180 degrees
- moved C1 293.4 mm to (343.4, 172.2), turned to 180 degrees
- moved C3 293.4 mm to (343.4, 169.2), turned to 180 degrees
- moved F1 292.3 mm to (342.9, 166.1), turned to 180 degrees
- moved D117 289.9 mm to (341.7, 143.3), turned to 180 degrees
- moved Y1 289.4 mm to (341.4, 159.6), turned to 180 degrees
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Other:
- outline, holes or cut-outs redrawn

Commit message: more pcb
Parts:
- removed D100, D101, D102, D103, D104, D105, D106, D107, D108, D109, D110, D111, D112, D113, D129, D130, D131, D132, D133, D134, D135, D136, D137, D138, D139, D140, D141, D142, D143, D144, D161, D162, D163, D164, D165, D166, D167, D168, D169, D170, D171, D99: D_Small, Diode_SMD:D_SOD-123
- removed D114: CapsLockRGB, LED_SMD:LED_SK6812MINI_PLCC4_3.5x3.5mm_P1.75mm
- removed D115: ARGB, LED_SMD:LED_SK6812MINI_PLCC4_3.5x3.5mm_P1.75mm
- removed D116: SRGB, LED_SMD:LED_SK6812MINI_PLCC4_3.5x3.5mm_P1.75mm
- removed D117: DRGB, LED_SMD:LED_SK6812MINI_PLCC4_3.5x3.5mm_P1.75mm
- removed D118: FRGB, LED_SMD:LED_SK6812MINI_PLCC4_3.5x3.5mm_P1.75mm
- removed D119: GRGB, LED_SMD:LED_SK6812MINI_PLCC4_3.5x3.5mm_P1.75mm
- removed D120: HRGB, LED_SMD:LED_SK6812MINI_PLCC4_3.5x3.5mm_P1.75mm
- removed D121: JRGB, LED_SMD:LED_SK6812MINI_PLCC4_3.5x3.5mm_P1.75mm
- removed D122: KRGB, LED_SMD:LED_SK6812MINI_PLCC4_3.5x3.5mm_P1.75mm
- removed D123: LRGB, LED_SMD:LED_SK6812MINI_PLCC4_3.5x3.5mm_P1.75mm
- removed D124: ;RGB, LED_SMD:LED_SK6812MINI_PLCC4_3.5x3.5mm_P1.75mm
- removed D125: '@RGB, LED_SMD:LED_SK6812MINI_PLCC4_3.5x3.5mm_P1.75mm
- removed D126: #~RGB, LED_SMD:LED_SK6812MINI_PLCC4_3.5x3.5mm_P1.75mm
- removed D127: HomeRGB, LED_SMD:LED_SK6812MINI_PLCC4_3.5x3.5mm_P1.75mm
- removed D128: EndRGB, LED_SMD:LED_SK6812MINI_PLCC4_3.5x3.5mm_P1.75mm
- removed D145: LShift, LED_SMD:LED_SK6812MINI_PLCC4_3.5x3.5mm_P1.75mm
- removed D146: \|RGB, LED_SMD:LED_SK6812MINI_PLCC4_3.5x3.5mm_P1.75mm
- removed D147: ZRGB, LED_SMD:LED_SK6812MINI_PLCC4_3.5x3.5mm_P1.75mm
- removed D148: XRGB, LED_SMD:LED_SK6812MINI_PLCC4_3.5x3.5mm_P1.75mm
- removed D149: CRGB, LED_SMD:LED_SK6812MINI_PLCC4_3.5x3.5mm_P1.75mm
- removed D150: VRGB, LED_SMD:LED_SK6812MINI_PLCC4_3.5x3.5mm_P1.75mm
- removed D151: BRGB, LED_SMD:LED_SK6812MINI_PLCC4_3.5x3.5mm_P1.75mm
- removed D152: NRGB, LED_SMD:LED_SK6812MINI_PLCC4_3.5x3.5mm_P1.75mm
- removed D153: MRGB, LED_SMD:LED_SK6812MINI_PLCC4_3.5x3.5mm_P1.75mm
- removed D154: ,<RGB, LED_SMD:LED_SK6812MINI_PLCC4_3.5x3.5mm_P1.75mm
- removed D155: .>RGB, LED_SMD:LED_SK6812MINI_PLCC4_3.5x3.5mm_P1.75mm
- removed D156: /?RGB, LED_SMD:LED_SK6812MINI_PLCC4_3.5x3.5mm_P1.75mm
- removed D157: RShiftRGB, LED_SMD:LED_SK6812MINI_PLCC4_3.5x3.5mm_P1.75mm
- removed D158: UpArrowRGB, LED_SMD:LED_SK6812MINI_PLCC4_3.5x3.5mm_P1.75mm
- removed D159: U2RGB, LED_SMD:LED_SK6812MINI_PLCC4_3.5x3.5mm_P1.75mm
- removed D160: U3RGB, LED_SMD:LED_SK6812MINI_PLCC4_3.5x3.5mm_P1.75mm
- removed D172: LCtrlRGB, LED_SMD:LED_SK6812MINI_PLCC4_3.5x3.5mm_P1.75mm
- removed D173: WinRGB, LED_SMD:LED_SK6812MINI_PLCC4_3.5x3.5mm_P1.75mm
- removed D174: AltRGB, LED_SMD:LED_SK6812MINI_PLCC4_3.5x3.5mm_P1.75mm
- removed D175: SpaceRGB, LED_SMD:LED_SK6812MINI_PLCC4_3.5x3.5mm_P1.75mm
- removed D176: AltGrRGB, LED_SMD:LED_SK6812MINI_PLCC4_3.5x3.5mm_P1.75mm
- removed D177: FnRGB, LED_SMD:LED_SK6812MINI_PLCC4_3.5x3.5mm_P1.75mm
- removed D178: RCtrlRGB, LED_SMD:LED_SK6812MINI_PLCC4_3.5x3.5mm_P1.75mm
- removed D179: LeftArrowRGB, LED_SMD:LED_SK6812MINI_PLCC4_3.5x3.5mm_P1.75mm
- removed D180: DownArrowRGB, LED_SMD:LED_SK6812MINI_PLCC4_3.5x3.5mm_P1.75mm
- removed D181: RightArrowRGB, LED_SMD:LED_SK6812MINI_PLCC4_3.5x3.5mm_P1.75mm
- removed D182: U4RGB, LED_SMD:LED_SK6812MINI_PLCC4_3.5x3.5mm_P1.75mm
- removed the D92 at (147.0, 42.4)
- removed D93: PRGB, LED_SMD:LED_SK6812MINI_PLCC4_3.5x3.5mm_P1.75mm
- removed D94: [RGB, LED_SMD:LED_SK6812MINI_PLCC4_3.5x3.5mm_P1.75mm
- removed D95: ]RGB, LED_SMD:LED_SK6812MINI_PLCC4_3.5x3.5mm_P1.75mm
- removed D96: EnterRGB, LED_SMD:LED_SK6812MINI_PLCC4_3.5x3.5mm_P1.75mm
- removed D97: DeleteRGB, LED_SMD:LED_SK6812MINI_PLCC4_3.5x3.5mm_P1.75mm
- removed D98: PgDnRGB, LED_SMD:LED_SK6812MINI_PLCC4_3.5x3.5mm_P1.75mm
- added LED1: MX_SK6812MINI-E, marbastlib-mx:LED_MX_6028R, B.Cu at (-90.5, -768.8)
- added LED10: MX_SK6812MINI-E, marbastlib-mx:LED_MX_6028R, B.Cu at (81.0, -768.8)
- added LED11: MX_SK6812MINI-E, marbastlib-mx:LED_MX_6028R, B.Cu at (100.0, -768.8)
- added LED12: MX_SK6812MINI-E, marbastlib-mx:LED_MX_6028R, B.Cu at (119.1, -768.8)
- added LED13: MX_SK6812MINI-E, marbastlib-mx:LED_MX_6028R, B.Cu at (138.1, -768.8)
- added LED14: MX_SK6812MINI-E, marbastlib-mx:LED_MX_6028R, B.Cu at (157.2, -768.8)
- added LED15: MX_SK6812MINI-E, marbastlib-mx:LED_MX_6028R, B.Cu at (176.2, -768.8)
- added LED16: MX_SK6812MINI-E, marbastlib-mx:LED_MX_6028R, B.Cu at (195.3, -768.8)
- added LED17: MX_SK6812MINI-E, marbastlib-mx:LED_MX_6028R, B.Cu at (214.3, -768.8)
- added LED18: MX_SK6812MINI-E, marbastlib-mx:LED_MX_6028R, B.Cu at (-90.5, -749.8)
- added LED19: MX_SK6812MINI-E, marbastlib-mx:LED_MX_6028R, B.Cu at (-71.4, -749.8)
- added LED2: MX_SK6812MINI-E, marbastlib-mx:LED_MX_6028R, B.Cu at (-71.4, -768.8)
- added LED20: MX_SK6812MINI-E, marbastlib-mx:LED_MX_6028R, B.Cu at (-52.4, -749.8)
- added LED21: MX_SK6812MINI-E, marbastlib-mx:LED_MX_6028R, B.Cu at (-33.3, -749.8)
- added LED22: MX_SK6812MINI-E, marbastlib-mx:LED_MX_6028R, B.Cu at (124.8, -308.9)
- added LED23: MX_SK6812MINI-E, marbastlib-mx:LED_MX_6028R, B.Cu at (-14.3, -749.8)
- added LED24: MX_SK6812MINI-E, marbastlib-mx:LED_MX_6028R, B.Cu at (4.76, -749.8)
- added LED25: MX_SK6812MINI-E, marbastlib-mx:LED_MX_6028R, B.Cu at (23.8, -749.8)
- added LED26: MX_SK6812MINI-E, marbastlib-mx:LED_MX_6028R, B.Cu at (42.8, -749.8)
- added LED27: MX_SK6812MINI-E, marbastlib-mx:LED_MX_6028R, B.Cu at (61.9, -749.8)
- added LED28: MX_SK6812MINI-E, marbastlib-mx:LED_MX_6028R, B.Cu at (81.0, -749.8)
- added LED29: MX_SK6812MINI-E, marbastlib-mx:LED_MX_6028R, B.Cu at (100.0, -749.8)
- added LED3: MX_SK6812MINI-E, marbastlib-mx:LED_MX_6028R, B.Cu at (-52.4, -768.8)
- added LED30: MX_SK6812MINI-E, marbastlib-mx:LED_MX_6028R, B.Cu at (119.1, -749.8)
- added LED31: MX_SK6812MINI-E, marbastlib-mx:LED_MX_6028R, B.Cu at (138.1, -749.8)
- added LED32: MX_SK6812MINI-E, marbastlib-mx:LED_MX_6028R, B.Cu at (166.7, -749.8)
- added LED33: MX_SK6812MINI-E, marbastlib-mx:LED_MX_6028R, B.Cu at (195.3, -749.8)
- added LED34: MX_SK6812MINI-E, marbastlib-mx:LED_MX_6028R, B.Cu at (214.3, -749.8)
- added LED35: MX_SK6812MINI-E, marbastlib-mx:LED_MX_6028R, B.Cu at (103.4, -207.9)
- added LED36: MX_SK6812MINI-E, marbastlib-mx:LED_MX_6028R, B.Cu at (184.2, -248.4)
- added LED37: MX_SK6812MINI-E, marbastlib-mx:LED_MX_6028R, B.Cu at (184.2, -147.4)
- added LED38: MX_SK6812MINI-E, marbastlib-mx:LED_MX_6028R, B.Cu at (164.0, -187.7)
- added LED39: MX_SK6812MINI-E, marbastlib-mx:LED_MX_6028R, B.Cu at (118.9, -288.7)
- added LED4: MX_SK6812MINI-E, marbastlib-mx:LED_MX_6028R, B.Cu at (-33.3, -768.8)
- added LED40: MX_SK6812MINI-E, marbastlib-mx:LED_MX_6028R, B.Cu at (164.0, -147.3)
- added LED41: MX_SK6812MINI-E, marbastlib-mx:LED_MX_6028R, B.Cu at (-36.8, -308.9)
- added LED42: MX_SK6812MINI-E, marbastlib-mx:LED_MX_6028R, B.Cu at (23.8, -308.9)
- added LED43: MX_SK6812MINI-E, marbastlib-mx:LED_MX_6028R, B.Cu at (78.5, -268.5)
- added LED44: MX_SK6812MINI-E, marbastlib-mx:LED_MX_6028R, B.Cu at (159.3, -288.7)
- added LED45: MX_SK6812MINI-E, marbastlib-mx:LED_MX_6028R, B.Cu at (78.5, -288.7)
- added LED46: MX_SK6812MINI-E, marbastlib-mx:LED_MX_6028R, B.Cu at (74.9, -329.1)
- added LED47: MX_SK6812MINI-E, marbastlib-mx:LED_MX_6028R, B.Cu at (184.2, -107.0)
- added LED48: MX_SK6812MINI-E, marbastlib-mx:LED_MX_6028R, B.Cu at (83.2, -187.7)
- added LED49: MX_SK6812MINI-E, marbastlib-mx:LED_MX_6028R, B.Cu at (123.6, -147.3)
- added LED5: MX_SK6812MINI-E, marbastlib-mx:LED_MX_6028R, B.Cu at (-14.3, -768.8)
- added LED50: MX_SK6812MINI-E, marbastlib-mx:LED_MX_6028R, B.Cu at (143.8, -187.7)
- added LED51: MX_SK6812MINI-E, marbastlib-mx:LED_MX_6028R, B.Cu at (95.1, -329.1)
- added LED52: MX_SK6812MINI-E, marbastlib-mx:LED_MX_6028R, B.Cu at (118.9, -268.5)
- added LED53: MX_SK6812MINI-E, marbastlib-mx:LED_MX_6028R, B.Cu at (14.3, -329.1)
- added LED54: MX_SK6812MINI-E, marbastlib-mx:LED_MX_6028R, B.Cu at (-46.3, -329.1)
- added LED55: MX_SK6812MINI-E, marbastlib-mx:LED_MX_6028R, B.Cu at (-22.5, -288.7)
- added LED56: MX_SK6812MINI-E, marbastlib-mx:LED_MX_6028R, B.Cu at (103.4, -228.1)
- added LED57: MX_SK6812MINI-E, marbastlib-mx:LED_MX_6028R, B.Cu at (123.6, -127.1)
- added LED58: MX_SK6812MINI-E, marbastlib-mx:LED_MX_6028R, B.Cu at (143.8, -106.9)
- added LED59: MX_SK6812MINI-E, marbastlib-mx:LED_MX_6028R, B.Cu at (-26.1, -329.1)
- added LED6: MX_SK6812MINI-E, marbastlib-mx:LED_MX_6028R, B.Cu at (4.76, -768.8)
- added LED60: MX_SK6812MINI-E, marbastlib-mx:LED_MX_6028R, B.Cu at (123.6, -248.3)
- added LED61: MX_SK6812MINI-E, marbastlib-mx:LED_MX_6028R, B.Cu at (-22.5, -268.5)
- added LED62: MX_SK6812MINI-E, marbastlib-mx:LED_MX_6028R, B.Cu at (143.8, -228.1)
- added LED63: MX_SK6812MINI-E, marbastlib-mx:LED_MX_6028R, B.Cu at (84.4, -308.9)
- added LED64: MX_SK6812MINI-E, marbastlib-mx:LED_MX_6028R, B.Cu at (83.2, -228.1)
- added LED65: MX_SK6812MINI-E, marbastlib-mx:LED_MX_6028R, B.Cu at (164.0, -228.1)
- added LED66: MX_SK6812MINI-E, marbastlib-mx:LED_MX_6028R, B.Cu at (164.0, -106.9)
- added LED67: MX_SK6812MINI-E, marbastlib-mx:LED_MX_6028R, B.Cu at (139.1, -288.7)
- added LED68: MX_SK6812MINI-E, marbastlib-mx:LED_MX_6028R, B.Cu at (58.3, -288.7)
- added LED69: MX_SK6812MINI-E, marbastlib-mx:LED_MX_6028R, B.Cu at (143.8, -147.3)
- added LED7: MX_SK6812MINI-E, marbastlib-mx:LED_MX_6028R, B.Cu at (23.8, -768.8)
- added LED70: MX_SK6812MINI-E, marbastlib-mx:LED_MX_6028R, B.Cu at (63.0, -187.7)
- added LED71: MX_SK6812MINI-E, marbastlib-mx:LED_MX_6028R, B.Cu at (-16.6, -308.9)
- added LED72: MX_SK6812MINI-E, marbastlib-mx:LED_MX_6028R, B.Cu at (164.0, -248.3)
- added LED73: MX_SK6812MINI-E, marbastlib-mx:LED_MX_6028R, B.Cu at (184.2, -127.2)
- added LED74: MX_SK6812MINI-E, marbastlib-mx:LED_MX_6028R, B.Cu at (-5.87, -329.1)
- added LED75: MX_SK6812MINI-E, marbastlib-mx:LED_MX_6028R, B.Cu at (63.0, -228.1)
- added LED76: MX_SK6812MINI-E, marbastlib-mx:LED_MX_6028R, B.Cu at (22.6, -228.1)
- added LED77: MX_SK6812MINI-E, marbastlib-mx:LED_MX_6028R, B.Cu at (83.2, -207.9)
- added LED78: MX_SK6812MINI-E, marbastlib-mx:LED_MX_6028R, B.Cu at (103.4, -167.5)
- added LED79: MX_SK6812MINI-E, marbastlib-mx:LED_MX_6028R, B.Cu at (54.7, -329.1)
- added LED8: MX_SK6812MINI-E, marbastlib-mx:LED_MX_6028R, B.Cu at (42.9, -768.8)
- added LED80: MX_SK6812MINI-E, marbastlib-mx:LED_MX_6028R, B.Cu at (34.5, -329.1)
- added LED81: MX_SK6812MINI-E, marbastlib-mx:LED_MX_6028R, B.Cu at (143.8, -248.3)
- added LED82: MX_SK6812MINI-E, marbastlib-mx:LED_MX_6028R, B.Cu at (103.4, -187.7)
- added LED83: MX_SK6812MINI-E, marbastlib-mx:LED_MX_6028R, B.Cu at (139.1, -268.5)
- added LED84: MX_SK6812MINI-E, marbastlib-mx:LED_MX_6028R, B.Cu at (64.2, -308.9)
- added LED85: MX_SK6812MINI-E, marbastlib-mx:LED_MX_6028R, B.Cu at (184.2, -167.6)
- added LED86: MX_SK6812MINI-E, marbastlib-mx:LED_MX_6028R, B.Cu at (38.1, -288.7)
- added LED87: MX_SK6812MINI-E, marbastlib-mx:LED_MX_6028R, B.Cu at (-66.5, -329.1)
- added LED88: MX_SK6812MINI-E, marbastlib-mx:LED_MX_6028R, B.Cu at (184.2, -228.2)
- added LED89: MX_SK6812MINI-E, marbastlib-mx:LED_MX_6028R, B.Cu at (3.62, -308.9)
- added LED9: MX_SK6812MINI-E, marbastlib-mx:LED_MX_6028R, B.Cu at (61.9, -768.8)
- added LED90: MX_SK6812MINI-E, marbastlib-mx:LED_MX_6028R, B.Cu at (164.0, -127.1)
- added LED91: MX_SK6812MINI-E, marbastlib-mx:LED_MX_6028R, B.Cu at (83.2, -248.3)
- D18: value ESCRGB -> D_Small; footprint LED_SMD:LED_SK6812MINI_PLCC4_3.5x3.5mm_P1.75mm -> Diode_SMD:D_SOD-123
- D19: value F1RGB -> D_Small; footprint LED_SMD:LED_SK6812MINI_PLCC4_3.5x3.5mm_P1.75mm -> Diode_SMD:D_SOD-123
- D20: value F2RGB -> D_Small; footprint LED_SMD:LED_SK6812MINI_PLCC4_3.5x3.5mm_P1.75mm -> Diode_SMD:D_SOD-123
- D21: value F3RGB -> D_Small; footprint LED_SMD:LED_SK6812MINI_PLCC4_3.5x3.5mm_P1.75mm -> Diode_SMD:D_SOD-123
- D22: value F4RGB -> D_Small; footprint LED_SMD:LED_SK6812MINI_PLCC4_3.5x3.5mm_P1.75mm -> Diode_SMD:D_SOD-123
- D23: value F5RGB -> D_Small; footprint LED_SMD:LED_SK6812MINI_PLCC4_3.5x3.5mm_P1.75mm -> Diode_SMD:D_SOD-123
- D24: value F6RGB -> D_Small; footprint LED_SMD:LED_SK6812MINI_PLCC4_3.5x3.5mm_P1.75mm -> Diode_SMD:D_SOD-123
- D25: value XEVRGB -> D_Small; footprint LED_SMD:LED_SK6812MINI_PLCC4_3.5x3.5mm_P1.75mm -> Diode_SMD:D_SOD-123
- D26: value F7RGB -> D_Small; footprint LED_SMD:LED_SK6812MINI_PLCC4_3.5x3.5mm_P1.75mm -> Diode_SMD:D_SOD-123
- D27: value F8RGB -> D_Small; footprint LED_SMD:LED_SK6812MINI_PLCC4_3.5x3.5mm_P1.75mm -> Diode_SMD:D_SOD-123
- D28: value F9RGB -> D_Small; footprint LED_SMD:LED_SK6812MINI_PLCC4_3.5x3.5mm_P1.75mm -> Diode_SMD:D_SOD-123
- D29: value F10RGB -> D_Small; footprint LED_SMD:LED_SK6812MINI_PLCC4_3.5x3.5mm_P1.75mm -> Diode_SMD:D_SOD-123
- D30: value F11RGB -> D_Small; footprint LED_SMD:LED_SK6812MINI_PLCC4_3.5x3.5mm_P1.75mm -> Diode_SMD:D_SOD-123
- D31: value F12RGB -> D_Small; footprint LED_SMD:LED_SK6812MINI_PLCC4_3.5x3.5mm_P1.75mm -> Diode_SMD:D_SOD-123
- D32: value U1RGB -> D_Small; footprint LED_SMD:LED_SK6812MINI_PLCC4_3.5x3.5mm_P1.75mm -> Diode_SMD:D_SOD-123
- D33: value PrtScRGB -> D_Small; footprint LED_SMD:LED_SK6812MINI_PLCC4_3.5x3.5mm_P1.75mm -> Diode_SMD:D_SOD-123
- D34: value PauseBrRGB -> D_Small; footprint LED_SMD:LED_SK6812MINI_PLCC4_3.5x3.5mm_P1.75mm -> Diode_SMD:D_SOD-123
- D51: value `RGB -> D_Small; footprint LED_SMD:LED_SK6812MINI_PLCC4_3.5x3.5mm_P1.75mm -> Diode_SMD:D_SOD-123
- D52: value 1RGB -> D_Small; footprint LED_SMD:LED_SK6812MINI_PLCC4_3.5x3.5mm_P1.75mm -> Diode_SMD:D_SOD-123
- D53: value 2RGB -> D_Small; footprint LED_SMD:LED_SK6812MINI_PLCC4_3.5x3.5mm_P1.75mm -> Diode_SMD:D_SOD-123
- D54: value 3RGB -> D_Small; footprint LED_SMD:LED_SK6812MINI_PLCC4_3.5x3.5mm_P1.75mm -> Diode_SMD:D_SOD-123
- D55: value 4RGB -> D_Small; footprint LED_SMD:LED_SK6812MINI_PLCC4_3.5x3.5mm_P1.75mm -> Diode_SMD:D_SOD-123
- D56: value 5RGB -> D_Small; footprint LED_SMD:LED_SK6812MINI_PLCC4_3.5x3.5mm_P1.75mm -> Diode_SMD:D_SOD-123
- D57: value 6RGB -> D_Small; footprint LED_SMD:LED_SK6812MINI_PLCC4_3.5x3.5mm_P1.75mm -> Diode_SMD:D_SOD-123
- D58: value 7RGB -> D_Small; footprint LED_SMD:LED_SK6812MINI_PLCC4_3.5x3.5mm_P1.75mm -> Diode_SMD:D_SOD-123
- D59: value 8RGB -> D_Small; footprint LED_SMD:LED_SK6812MINI_PLCC4_3.5x3.5mm_P1.75mm -> Diode_SMD:D_SOD-123
- D60: value 9RGB -> D_Small; footprint LED_SMD:LED_SK6812MINI_PLCC4_3.5x3.5mm_P1.75mm -> Diode_SMD:D_SOD-123
- D61: value 0RGB -> D_Small; footprint LED_SMD:LED_SK6812MINI_PLCC4_3.5x3.5mm_P1.75mm -> Diode_SMD:D_SOD-123
- D62: value -RGB -> D_Small; footprint LED_SMD:LED_SK6812MINI_PLCC4_3.5x3.5mm_P1.75mm -> Diode_SMD:D_SOD-123
- D63: value =RGB -> D_Small; footprint LED_SMD:LED_SK6812MINI_PLCC4_3.5x3.5mm_P1.75mm -> Diode_SMD:D_SOD-123
- D64: value BackSpaceRGB -> D_Small; footprint LED_SMD:LED_SK6812MINI_PLCC4_3.5x3.5mm_P1.75mm -> Diode_SMD:D_SOD-123
- D65: value InsertRGB -> D_Small; footprint LED_SMD:LED_SK6812MINI_PLCC4_3.5x3.5mm_P1.75mm -> Diode_SMD:D_SOD-123
- D66: value PgUpRGB -> D_Small; footprint LED_SMD:LED_SK6812MINI_PLCC4_3.5x3.5mm_P1.75mm -> Diode_SMD:D_SOD-123
- D83: value TabRGB -> D_Small; footprint LED_SMD:LED_SK6812MINI_PLCC4_3.5x3.5mm_P1.75mm -> Diode_SMD:D_SOD-123
- D84: value QRGB -> D_Small; footprint LED_SMD:LED_SK6812MINI_PLCC4_3.5x3.5mm_P1.75mm -> Diode_SMD:D_SOD-123
- D85: value WRGB -> D_Small; footprint LED_SMD:LED_SK6812MINI_PLCC4_3.5x3.5mm_P1.75mm -> Diode_SMD:D_SOD-123
- D86: value ERGB -> D_Small; footprint LED_SMD:LED_SK6812MINI_PLCC4_3.5x3.5mm_P1.75mm -> Diode_SMD:D_SOD-123
- D87: value RRGB -> D_Small; footprint LED_SMD:LED_SK6812MINI_PLCC4_3.5x3.5mm_P1.75mm -> Diode_SMD:D_SOD-123
- D88: value TRGB -> D_Small; footprint LED_SMD:LED_SK6812MINI_PLCC4_3.5x3.5mm_P1.75mm -> Diode_SMD:D_SOD-123
- D89: value YRGB -> D_Small; footprint LED_SMD:LED_SK6812MINI_PLCC4_3.5x3.5mm_P1.75mm -> Diode_SMD:D_SOD-123
- D90: value URGB -> D_Small; footprint LED_SMD:LED_SK6812MINI_PLCC4_3.5x3.5mm_P1.75mm -> Diode_SMD:D_SOD-123
- D91: value IRGB -> D_Small; footprint LED_SMD:LED_SK6812MINI_PLCC4_3.5x3.5mm_P1.75mm -> Diode_SMD:D_SOD-123
- SW1: value ESC -> Esc
- SW10: value F8 -> #F8
- SW11: value F9 -> #F9
- SW12: value F10 -> #F10
- SW13: value F11 -> #F11
- SW14: value F12 -> #F12
- SW15: value U1 -> U5
- SW17: value PauseBr -> PauseBreak
- SW2: value F1 -> #F1
- SW3: value F2 -> #F2
- SW37: value E -> #E
- SW38: value R -> #R
- SW4: value F3 -> #F3
- SW5: value F4 -> #F4
- SW51: value A -> #A
- SW53: value D -> #D
- SW54: value F -> #F
- SW6: value F5 -> #F5
- SW60: value ; -> ;:
- SW62: value #~ -> ~#
- SW69: value C -> #C
- SW7: value F6 -> #F6
- SW9: value F7 -> #F7
- moved D63 655.4 mm to (-188.2, -302.3)
- moved D59 634.6 mm to (-176.7, -298.9)
- moved D37 620.0 mm to (-226.4, -339.2)
- moved D24 608.2 mm to (-188.2, -298.9)
- moved D34 604.0 mm to (-220.6, -335.9)
- moved D45 586.4 mm to (-182.4, -302.3)
- moved D38 575.8 mm to (-226.4, -342.6)
- moved D14 571.3 mm to (-211.1, -322.4)
- moved REF** 562.8 mm to (166.7, -754.9)
- moved SW18 562.8 mm to (-90.5, -754.9)
- moved SW19 562.8 mm to (-71.4, -754.9)
- moved SW20 562.8 mm to (-52.4, -754.9)
- moved SW21 562.8 mm to (-33.3, -754.9)
- moved SW22 562.8 mm to (-14.3, -754.9)
- moved SW23 562.8 mm to (4.76, -754.9)
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- renumbered D183 to D92
Connections:
- D18 pad 1: Net-(D18-Pad1) -> row1
- D18 pad 2: GND -> Net-(D18-Pad2)
- D19 pad 1: Net-(D19-Pad1) -> row1
- D19 pad 2: GND -> Net-(D19-Pad2)
- D20 pad 1: Net-(D20-Pad1) -> row1
- D20 pad 2: GND -> Net-(D20-Pad2)
- D21 pad 1: Net-(D21-Pad1) -> row1
- D21 pad 2: GND -> Net-(D21-Pad2)
- D22 pad 1: Net-(D22-Pad1) -> row1
- D22 pad 2: GND -> Net-(D22-Pad2)
- D23 pad 1: Net-(D23-Pad1) -> row1
- D23 pad 2: GND -> Net-(D23-Pad2)
- D24 pad 1: Net-(D24-Pad1) -> row1
- D24 pad 2: GND -> Net-(D24-Pad2)
- D25 pad 1: Net-(D25-Pad1) -> row1
- D25 pad 2: GND -> Net-(D25-Pad2)
- D26 pad 1: Net-(D26-Pad1) -> row1
- D26 pad 2: GND -> Net-(D26-Pad2)
- D27 pad 1: Net-(D27-Pad1) -> row1
- D27 pad 2: GND -> Net-(D27-Pad2)
- D28 pad 1: Net-(D28-Pad1) -> row1
- D28 pad 2: GND -> Net-(D28-Pad2)
- D29 pad 1: Net-(D29-Pad1) -> row1
- D29 pad 2: GND -> Net-(D29-Pad2)
- D30 pad 1: Net-(D30-Pad1) -> row1
- D30 pad 2: GND -> Net-(D30-Pad2)
- D31 pad 1: Net-(D31-Pad1) -> row1
- D31 pad 2: GND -> Net-(D31-Pad2)
- D32 pad 1: Net-(D32-Pad1) -> row1
- D32 pad 2: GND -> Net-(D32-Pad2)
- D33 pad 1: Net-(D33-Pad1) -> row1
- D33 pad 2: GND -> Net-(D33-Pad2)
- D34 pad 1: Net-(D34-Pad1) -> row2
- D34 pad 2: GND -> Net-(D34-Pad2)
- D35 pad 1: row1 -> row2
- D36 pad 1: row1 -> row2
- D37 pad 1: row1 -> row2
- D38 pad 1: row1 -> row2
- D39 pad 1: row1 -> row2
- D40 pad 1: row1 -> row2
- D41 pad 1: row1 -> row2
- D42 pad 1: row1 -> row2
- D43 pad 1: row1 -> row2
- D44 pad 1: row1 -> row2
- D45 pad 1: row1 -> row2
- D46 pad 1: row1 -> row2
- D47 pad 1: row1 -> row2
- D48 pad 1: row1 -> row2
- D49 pad 1: row1 -> row2
- D50 pad 1: row1 -> row3
- D51 pad 1: Net-(D51-Pad1) -> row3
- D51 pad 2: GND -> Net-(D51-Pad2)
- D52 pad 1: Net-(D52-Pad1) -> row3
- D52 pad 2: GND -> Net-(D52-Pad2)
- D53 pad 1: Net-(D53-Pad1) -> row3
- D53 pad 2: GND -> Net-(D53-Pad2)
- D54 pad 1: Net-(D54-Pad1) -> row3
- D54 pad 2: GND -> Net-(D54-Pad2)
- D55 pad 1: Net-(D55-Pad1) -> row3
- D55 pad 2: GND -> Net-(D55-Pad2)
- D56 pad 1: Net-(D56-Pad1) -> row3
- D56 pad 2: GND -> Net-(D56-Pad2)
- D57 pad 1: Net-(D57-Pad1) -> row3
- D57 pad 2: GND -> Net-(D57-Pad2)
- D58 pad 1: Net-(D58-Pad1) -> row3
- D58 pad 2: GND -> Net-(D58-Pad2)
- D59 pad 1: Net-(D59-Pad1) -> row3
- D59 pad 2: GND -> Net-(D59-Pad2)
- D60 pad 1: Net-(D60-Pad1) -> row3
- D60 pad 2: GND -> Net-(D60-Pad2)
- D61 pad 1: Net-(D61-Pad1) -> row3
- D61 pad 2: GND -> Net-(D61-Pad2)
- D62 pad 1: Net-(D62-Pad1) -> row3
- D62 pad 2: GND -> Net-(D62-Pad2)
- D63 pad 1: Net-(D63-Pad1) -> row3
- D63 pad 2: GND -> Net-(D63-Pad2)
- D64 pad 1: Net-(D64-Pad1) -> row3
- D64 pad 2: GND -> Net-(D64-Pad2)
- D65 pad 1: Net-(D65-Pad1) -> row4
- D65 pad 2: GND -> Net-(D65-Pad2)
- D66 pad 1: Net-(D66-Pad1) -> row4
- D66 pad 2: GND -> Net-(D66-Pad2)
- D67 pad 1: row2 -> row4
- D68 pad 1: row2 -> row4
- D69 pad 1: row2 -> row4
- D70 pad 1: row2 -> row4
- D71 pad 1: row2 -> row4
- D72 pad 1: row2 -> row4
- D73 pad 1: row2 -> row4
- D74 pad 1: row2 -> row4
- D75 pad 1: row2 -> row4
- D76 pad 1: row2 -> row4
- D77 pad 1: row2 -> row4
- D78 pad 1: row2 -> row4
- D79 pad 1: row2 -> row4
- D80 pad 1: row2 -> row4
- D81 pad 1: row2 -> row5
- D82 pad 1: row2 -> row5
- D83 pad 1: Net-(D83-Pad1) -> row5
- D83 pad 2: GND -> Net-(D83-Pad2)
- D84 pad 1: Net-(D84-Pad1) -> row5
- D84 pad 2: GND -> Net-(D84-Pad2)
- D85 pad 1: Net-(D85-Pad1) -> row5
- D85 pad 2: GND -> Net-(D85-Pad2)
- D86 pad 1: Net-(D86-Pad1) -> row5
- D86 pad 2: GND -> Net-(D86-Pad2)
- D87 pad 1: Net-(D87-Pad1) -> row5
- D87 pad 2: GND -> Net-(D87-Pad2)
- D88 pad 1: Net-(D88-Pad1) -> row5
- D88 pad 2: GND -> Net-(D88-Pad2)
- D89 pad 1: Net-(D89-Pad1) -> row5
- D89 pad 2: GND -> Net-(D89-Pad2)
- D90 pad 1: Net-(D90-Pad1) -> row5
- D90 pad 2: GND -> Net-(D90-Pad2)
- D91 pad 1: Net-(D91-Pad1) -> row5
- D91 pad 2: GND -> Net-(D91-Pad2)
- SW1 pad 1: Net-(D1-Pad2) -> col0
- SW1 pad 2: col0 -> Net-(D1-Pad2)
- SW10 pad 1: Net-(D10-Pad2) -> col9
- SW10 pad 2: col9 -> Net-(D10-Pad2)
- SW11 pad 1: Net-(D11-Pad2) -> col10
- SW11 pad 2: col10 -> Net-(D11-Pad2)
- SW12 pad 1: Net-(D12-Pad2) -> col11
- SW12 pad 2: col11 -> Net-(D12-Pad2)
- SW13 pad 1: Net-(D13-Pad2) -> col12
- SW13 pad 2: col12 -> Net-(D13-Pad2)
- SW14 pad 1: Net-(D14-Pad2) -> col13
- SW14 pad 2: col13 -> Net-(D14-Pad2)
- SW15 pad 1: Net-(D15-Pad2) -> col14
- SW15 pad 2: col14 -> Net-(D15-Pad2)
- SW16 pad 1: Net-(D16-Pad2) -> col15
- SW16 pad 2: col15 -> Net-(D16-Pad2)
- SW17 pad 1: Net-(D17-Pad2) -> MISO
- SW17 pad 2: MISO -> Net-(D17-Pad2)
- SW18 pad 1: Net-(D35-Pad2) -> col0
- SW18 pad 2: col0 -> Net-(D18-Pad2)
- SW19 pad 1: Net-(D36-Pad2) -> col1
- SW19 pad 2: col1 -> Net-(D19-Pad2)
- SW2 pad 1: Net-(D2-Pad2) -> col1
- SW2 pad 2: col1 -> Net-(D2-Pad2)
- SW20 pad 1: Net-(D37-Pad2) -> col2
- SW20 pad 2: col2 -> Net-(D20-Pad2)
- SW21 pad 1: Net-(D38-Pad2) -> col3
- SW21 pad 2: col3 -> Net-(D21-Pad2)
- SW22 pad 1: Net-(D39-Pad2) -> col4
- SW22 pad 2: col4 -> Net-(D22-Pad2)
- SW23 pad 1: Net-(D40-Pad2) -> col5
- SW23 pad 2: col5 -> Net-(D23-Pad2)
- SW24 pad 1: Net-(D41-Pad2) -> col6
- SW24 pad 2: col6 -> Net-(D24-Pad2)
- SW25 pad 1: Net-(D42-Pad2) -> col7
- SW25 pad 2: col7 -> Net-(D25-Pad2)
- SW26 pad 1: Net-(D43-Pad2) -> col8
- SW26 pad 2: col8 -> Net-(D26-Pad2)
- SW27 pad 1: Net-(D44-Pad2) -> col9
- SW27 pad 2: col9 -> Net-(D27-Pad2)
- SW28 pad 1: Net-(D45-Pad2) -> col10
- SW28 pad 2: col10 -> Net-(D28-Pad2)
- SW29 pad 1: Net-(D46-Pad2) -> col11
- SW29 pad 2: col11 -> Net-(D29-Pad2)
- SW3 pad 1: Net-(D3-Pad2) -> col2
- SW3 pad 2: col2 -> Net-(D3-Pad2)
- SW30 pad 1: Net-(D47-Pad2) -> col12
- SW30 pad 2: col12 -> Net-(D30-Pad2)
- SW31 pad 1: Net-(D48-Pad2) -> col13
- SW31 pad 2: col13 -> Net-(D31-Pad2)
- SW32 pad 1: Net-(D49-Pad2) -> col15
- SW32 pad 2: col15 -> Net-(D32-Pad2)
- SW33 pad 1: Net-(D50-Pad2) -> MISO
- SW33 pad 2: MISO -> Net-(D33-Pad2)
- SW34 pad 1: Net-(D67-Pad2) -> col0
- SW34 pad 2: col0 -> Net-(D34-Pad2)
- SW35 pad 1: Net-(D68-Pad2) -> col1
- SW35 pad 2: col1 -> Net-(D35-Pad2)
- SW36 pad 1: Net-(D69-Pad2) -> col2
- SW36 pad 2: col2 -> Net-(D36-Pad2)
- SW37 pad 1: Net-(D70-Pad2) -> col3
- SW37 pad 2: col3 -> Net-(D37-Pad2)
- SW38 pad 1: Net-(D71-Pad2) -> col4
- SW38 pad 2: col4 -> Net-(D38-Pad2)
- SW39 pad 1: Net-(D72-Pad2) -> col5
- SW39 pad 2: col5 -> Net-(D39-Pad2)
- SW4 pad 1: Net-(D4-Pad2) -> col3
- SW4 pad 2: col3 -> Net-(D4-Pad2)
- SW40 pad 1: Net-(D73-Pad2) -> col6
- SW40 pad 2: col6 -> Net-(D40-Pad2)
- SW41 pad 1: Net-(D74-Pad2) -> col7
- SW41 pad 2: col7 -> Net-(D41-Pad2)
- SW42 pad 1: Net-(D75-Pad2) -> col8
- SW42 pad 2: col8 -> Net-(D42-Pad2)
- SW43 pad 1: Net-(D76-Pad2) -> col9
- SW43 pad 2: col9 -> Net-(D43-Pad2)
- SW44 pad 1: Net-(D77-Pad2) -> col10
- SW44 pad 2: col10 -> Net-(D44-Pad2)
- SW45 pad 1: Net-(D78-Pad2) -> col11
- SW45 pad 2: col11 -> Net-(D45-Pad2)
- SW46 pad 1: Net-(D79-Pad2) -> col12
- SW46 pad 2: col12 -> Net-(D46-Pad2)
- SW47 pad 1: Net-(D80-Pad2) -> col13
- SW47 pad 2: col13 -> Net-(D47-Pad2)
- SW48 pad 1: Net-(D81-Pad2) -> col15
- SW48 pad 2: col15 -> Net-(D48-Pad2)
- SW49 pad 1: Net-(D82-Pad2) -> MISO
- SW49 pad 2: MISO -> Net-(D49-Pad2)
- SW5 pad 1: Net-(D5-Pad2) -> col4
- SW5 pad 2: col4 -> Net-(D5-Pad2)
- SW50 pad 1: Net-(D99-Pad2) -> col0
- SW50 pad 2: col0 -> Net-(D50-Pad2)
- SW51 pad 1: Net-(D100-Pad2) -> col1
- SW51 pad 2: col1 -> Net-(D51-Pad2)
- SW52 pad 1: Net-(D101-Pad2) -> col2
- SW52 pad 2: col2 -> Net-(D52-Pad2)
- SW53 pad 1: Net-(D102-Pad2) -> col3
- SW53 pad 2: col3 -> Net-(D53-Pad2)
- SW54 pad 1: Net-(D103-Pad2) -> col4
- SW54 pad 2: col4 -> Net-(D54-Pad2)
- SW55 pad 1: Net-(D104-Pad2) -> col5
- SW55 pad 2: col5 -> Net-(D55-Pad2)
- SW56 pad 1: Net-(D105-Pad2) -> col6
- SW56 pad 2: col6 -> Net-(D56-Pad2)
- SW57 pad 1: Net-(D106-Pad2) -> col7
- SW57 pad 2: col7 -> Net-(D57-Pad2)
- SW58 pad 1: Net-(D107-Pad2) -> col8
- SW58 pad 2: col8 -> Net-(D58-Pad2)
- SW59 pad 1: Net-(D108-Pad2) -> col9
- SW59 pad 2: col9 -> Net-(D59-Pad2)
- SW6 pad 1: Net-(D6-Pad2) -> col5
- SW6 pad 2: col5 -> Net-(D6-Pad2)
- SW60 pad 1: Net-(D109-Pad2) -> col10
- SW60 pad 2: col10 -> Net-(D60-Pad2)
- SW61 pad 1: Net-(D110-Pad2) -> col11
- SW61 pad 2: col11 -> Net-(D61-Pad2)
- SW62 pad 1: Net-(D111-Pad2) -> col12
- SW62 pad 2: col12 -> Net-(D62-Pad2)
- SW63 pad 1: Net-(D112-Pad2) -> col15
- SW63 pad 2: col15 -> Net-(D63-Pad2)
- SW64 pad 1: Net-(D113-Pad2) -> MISO
- SW64 pad 2: MISO -> Net-(D64-Pad2)
- SW65 pad 1: Net-(D129-Pad2) -> col0
- SW65 pad 2: col0 -> Net-(D65-Pad2)
- SW66 pad 1: Net-(D130-Pad2) -> col1
- SW66 pad 2: col1 -> Net-(D66-Pad2)
- SW67 pad 1: Net-(D131-Pad2) -> col2
- SW67 pad 2: col2 -> Net-(D67-Pad2)
- SW68 pad 1: Net-(D132-Pad2) -> col3
- SW68 pad 2: col3 -> Net-(D68-Pad2)
- SW69 pad 1: Net-(D133-Pad2) -> col4
- SW69 pad 2: col4 -> Net-(D69-Pad2)
- SW7 pad 1: Net-(D7-Pad2) -> col6
- SW7 pad 2: col6 -> Net-(D7-Pad2)
- SW70 pad 1: Net-(D134-Pad2) -> col5
- SW70 pad 2: col5 -> Net-(D70-Pad2)
- SW71 pad 1: Net-(D135-Pad2) -> col6
- SW71 pad 2: col6 -> Net-(D71-Pad2)
- SW72 pad 1: Net-(D136-Pad2) -> col7
- SW72 pad 2: col7 -> Net-(D72-Pad2)
- SW73 pad 1: Net-(D137-Pad2) -> col8
- SW73 pad 2: col8 -> Net-(D73-Pad2)
- SW74 pad 1: Net-(D138-Pad2) -> col9
- SW74 pad 2: col9 -> Net-(D74-Pad2)
- SW75 pad 1: Net-(D139-Pad2) -> col10
- SW75 pad 2: col10 -> Net-(D75-Pad2)
- SW76 pad 1: Net-(D140-Pad2) -> col11
- SW76 pad 2: col11 -> Net-(D76-Pad2)
- SW77 pad 1: Net-(D141-Pad2) -> col12
- SW77 pad 2: col12 -> Net-(D77-Pad2)
- SW78 pad 1: Net-(D142-Pad2) -> col13
- SW78 pad 2: col13 -> Net-(D78-Pad2)
- SW79 pad 1: Net-(D143-Pad2) -> col15
- SW79 pad 2: col15 -> Net-(D79-Pad2)
- SW8 pad 1: Net-(D8-Pad2) -> col7
- SW8 pad 2: col7 -> Net-(D8-Pad2)
- SW80 pad 1: Net-(D144-Pad2) -> MISO
- SW80 pad 2: MISO -> Net-(D80-Pad2)
- SW81 pad 1: Net-(D161-Pad2) -> col0
- SW81 pad 2: col0 -> Net-(D81-Pad2)
- SW82 pad 1: Net-(D162-Pad2) -> col1
- SW82 pad 2: col1 -> Net-(D82-Pad2)
- SW83 pad 1: Net-(D163-Pad2) -> col2
- SW83 pad 2: col2 -> Net-(D83-Pad2)
- SW84 pad 1: Net-(D164-Pad2) -> col6
- SW84 pad 2: col6 -> Net-(D84-Pad2)
- SW85 pad 1: Net-(D165-Pad2) -> col10
- SW85 pad 2: col10 -> Net-(D85-Pad2)
- SW86 pad 1: Net-(D166-Pad2) -> col11
- SW86 pad 2: col11 -> Net-(D86-Pad2)
- SW87 pad 1: Net-(D167-Pad2) -> col12
- SW87 pad 2: col12 -> Net-(D87-Pad2)
- SW88 pad 1: Net-(D168-Pad2) -> col13
- SW88 pad 2: col13 -> Net-(D88-Pad2)
- SW89 pad 1: Net-(D169-Pad2) -> col14
- SW89 pad 2: col14 -> Net-(D89-Pad2)
- SW9 pad 1: Net-(D9-Pad2) -> col8
- SW9 pad 2: col8 -> Net-(D9-Pad2)
- SW90 pad 1: Net-(D170-Pad2) -> col15
- SW90 pad 2: col15 -> Net-(D90-Pad2)
- SW91 pad 1: Net-(D171-Pad2) -> MISO
- SW91 pad 2: MISO -> Net-(D91-Pad2)
Other:
- outline, holes or cut-outs redrawn
